File: hw/pwr_supply_sheet.sch (KiCad schematic (older format))
At the start: 15 parts

Commit message: CM_6.2.1 delivered, first customer machine with CCU, HCU & ICU
Parts:
- C201, C205: symbol icu-rescue:100nF -> 100nF
- C202: symbol icu-rescue:CAP_EEE-FK1H470P -> CAP_EEE-FK1H470P
- C203: symbol icu-rescue:10nF -> 10nF
- C204: symbol icu-rescue:T491D226K035AT -> T491D226K035AT
- D201, D206: symbol icu-rescue:DIODE_RS07J-GS18 -> DIODE_RS07J-GS18
- D202, D203: symbol icu-rescue:SCHOTTKY_DIODE_V40PW10C -> SCHOTTKY_DIODE_V40PW10C
- D204: symbol icu-rescue:DIODE_TVS_SMBJ33A-TRDO-214AA -> DIODE_TVS_SMBJ33A-TRDO-214AA
- D205: symbol icu-rescue:DIODE_TVS_TPSMD28A -> DIODE_TVS_TPSMD28A
- F201: symbol icu-rescue:FUSE_MC36211_350MA -> FUSE_MC36211_350MA
- L201: symbol icu-rescue:IND_744045210 -> IND_744045210
- VR201: symbol icu-rescue:LM2671SOIC8 -> LM2671SOIC8
- VR202: symbol icu-rescue:REG_MCP1700 -> REG_MCP1700
Changed lines of the file:
@@
-EESchema Schematic File Version 4
+EESchema Schematic File Version 2
+LIBS:kemet
+LIBS:usevolt
+LIBS:wurth_elektronik_LED
+LIBS:power
+LIBS:yageo
 LIBS:icu-cache
 EELAYER 26 0
@@
 $Descr A4 11693 8268
 encoding utf-8
-Sheet 2 13
+Sheet 2 14
 Title "Power supply"
 Date "2016-08-20"
@@
 VIN
 $Comp
-L icu-rescue:FUSE_MC36211_350MA F201
+L FUSE_MC36211_350MA F201
 U 1 1 57B8204F
 P 2500 3850
@@
 $EndComp
 $Comp
-L icu-rescue:DIODE_TVS_SMBJ33A-TRDO-214AA D204
+L DIODE_TVS_SMBJ33A-TRDO-214AA D204
 U 1 1 57B820C1
 P 2800 4050
@@
 $EndComp
 $Comp
-L icu-rescue:100nF C201
+L 100nF C201
 U 1 1 57B8217A
 P 3400 3950
@@
 $EndComp
 $Comp
-L icu-rescue:LM2671SOIC8 VR?
+L LM2671SOIC8 VR?
 U 1 1 57B82261
 P 4850 4150
@@
 $EndComp
 $Comp
-L icu-rescue:10nF C203
+L 10nF C203
 U 1 1 57B822C5
 P 5800 3950
@@
 $EndComp
 $Comp
-L icu-rescue:DIODE_RS07J-GS18 D206
+L DIODE_RS07J-GS18 D206
 U 1 1 57B82329
 P 6200 3950
@@
 $EndComp
 $Comp
-L icu-rescue:100nF C205
+L 100nF C205
 U 1 1 57B82A3F
 P 8600 3950
@@
 $EndComp
 $Comp
-L icu-rescue:+5V #PWR05
+L +5V #PWR05
 U 1 1 57B831F8
 P 6850 3600
@@
 $EndComp
 $Comp
-L icu-rescue:+3V3 #PWR06
+L +3V3 #PWR06
 U 1 1 57B83259
 P 8600 3600
@@
 NoConn ~ 4550 4050
 $Comp
-L icu-rescue:VDD #PWR07
+L VDD #PWR07
 U 1 1 57B9C56A
 P 3800 2100
@@
 $EndComp
 $Comp
-L icu-rescue:PWR_FLAG #FLG08
+L PWR_FLAG #FLG08
 U 1 1 57B9C59C
 P 3800 2300
@@
 $EndComp
 $Comp
-L icu-rescue:GND #PWR09
+L GND #PWR09
 U 1 1 57B9D351
 P 4300 2350
@@
 $EndComp
 $Comp
-L icu-rescue:PWR_FLAG #FLG010
+L PWR_FLAG #FLG010
 U 1 1 57B9D3A1
 P 4300 2150
@@
 $EndComp
 $Comp
-L icu-rescue:GND #PWR011
+L GND #PWR011
 U 1 1 57CF1F5E
 P 2800 5150
@@
 $EndComp
 $Comp
-L icu-rescue:IND_744045210 L201
+L IND_744045210 L201
 U 1 1 58945E39
 P 6500 3850
@@
 $EndComp
 $Comp
-L icu-rescue:DIODE_RS07J-GS18 D201
+L DIODE_RS07J-GS18 D201
 U 1 1 5896E2A2
 P 1900 3850
@@
 $EndComp
 $Comp
-L icu-rescue:T491D226K035AT C204
+L T491D226K035AT C204
 U 1 1 597AF606
 P 6850 4050
@@
 $EndComp
 $Comp
-L icu-rescue:REG_MCP1700 VR202
+L REG_MCP1700 VR202
 U 1 1 597AF83E
 P 8000 3950
@@
 $EndComp
 $Comp
-L icu-rescue:SCHOTTKY_DIODE_V40PW10C D203
+L SCHOTTKY_DIODE_V40PW10C D203
 U 1 1 59B7B8B2
 P 2050 3250
@@
 $EndComp
 $Comp
-L icu-rescue:SCHOTTKY_DIODE_V40PW10C D202
+L SCHOTTKY_DIODE_V40PW10C D202
 U 1 1 59D9089A
 P 2050 2750
@@
 $EndComp
 $Comp
-L icu-rescue:CAP_EEE-FK1H470P C202
+L CAP_EEE-FK1H470P C202
 U 1 1 5A13B69C
 P 3800 4050
@@
 $EndComp
 $Comp
-L icu-rescue:DIODE_TVS_TPSMD28A D205
+L DIODE_TVS_TPSMD28A D205
 U 1 1 5A13BC8E
 P 2900 2950
@@
 $EndComp
 $Comp
-L icu-rescue:GND #PWR012
+L GND #PWR012
 U 1 1 5A13BD77
 P 2900 3150

Commit message: 050518: Kikepera head prototype first revision, saw not working
Parts:
- C201, C205: symbol 100nF -> icu-rescue:100nF
- C202: symbol CAP_EEE-FK1H470P -> icu-rescue:CAP_EEE-FK1H470P
- C203: symbol 10nF -> icu-rescue:10nF
- C204: symbol T491D226K035AT -> icu-rescue:T491D226K035AT
- D201, D206: symbol DIODE_RS07J-GS18 -> icu-rescue:DIODE_RS07J-GS18
- D202, D203: symbol SCHOTTKY_DIODE_V40PW10C -> icu-rescue:SCHOTTKY_DIODE_V40PW10C
- D204: symbol DIODE_TVS_SMBJ33A-TRDO-214AA -> icu-rescue:DIODE_TVS_SMBJ33A-TRDO-214AA
- D205: symbol DIODE_TVS_TPSMD28A -> icu-rescue:DIODE_TVS_TPSMD28A
- F201: symbol FUSE_MC36211_350MA -> icu-rescue:FUSE_MC36211_350MA
- L201: symbol IND_744045210 -> icu-rescue:IND_744045210
- VR201: symbol LM2671SOIC8 -> icu-rescue:LM2671SOIC8
- VR202: symbol REG_MCP1700 -> icu-rescue:REG_MCP1700
Changed lines of the file:
@@
-EESchema Schematic File Version 2
-LIBS:kemet
-LIBS:usevolt
-LIBS:wurth_elektronik_LED
-LIBS:power
-LIBS:yageo
+EESchema Schematic File Version 4
 LIBS:icu-cache
 EELAYER 26 0
@@
 VIN
 $Comp
-L FUSE_MC36211_350MA F201
+L icu-rescue:FUSE_MC36211_350MA F201
 U 1 1 57B8204F
 P 2500 3850
@@
 $EndComp
 $Comp
-L DIODE_TVS_SMBJ33A-TRDO-214AA D204
+L icu-rescue:DIODE_TVS_SMBJ33A-TRDO-214AA D204
 U 1 1 57B820C1
 P 2800 4050
@@
 $EndComp
 $Comp
-L 100nF C201
+L icu-rescue:100nF C201
 U 1 1 57B8217A
 P 3400 3950
@@
 $EndComp
 $Comp
-L LM2671SOIC8 VR?
+L icu-rescue:LM2671SOIC8 VR?
 U 1 1 57B82261
 P 4850 4150
@@
 $EndComp
 $Comp
-L 10nF C203
+L icu-rescue:10nF C203
 U 1 1 57B822C5
 P 5800 3950
@@
 $EndComp
 $Comp
-L DIODE_RS07J-GS18 D206
+L icu-rescue:DIODE_RS07J-GS18 D206
 U 1 1 57B82329
 P 6200 3950
@@
 $EndComp
 $Comp
-L 100nF C205
+L icu-rescue:100nF C205
 U 1 1 57B82A3F
 P 8600 3950
@@
 $EndComp
 $Comp
-L +5V #PWR05
+L icu-rescue:+5V #PWR05
 U 1 1 57B831F8
 P 6850 3600
@@
 $EndComp
 $Comp
-L +3V3 #PWR06
+L icu-rescue:+3V3 #PWR06
 U 1 1 57B83259
 P 8600 3600
@@
 NoConn ~ 4550 4050
 $Comp
-L VDD #PWR07
+L icu-rescue:VDD #PWR07
 U 1 1 57B9C56A
 P 3800 2100
@@
 $EndComp
 $Comp
-L PWR_FLAG #FLG08
+L icu-rescue:PWR_FLAG #FLG08
 U 1 1 57B9C59C
 P 3800 2300
@@
 $EndComp
 $Comp
-L GND #PWR09
+L icu-rescue:GND #PWR09
 U 1 1 57B9D351
 P 4300 2350
@@
 $EndComp
 $Comp
-L PWR_FLAG #FLG010
+L icu-rescue:PWR_FLAG #FLG010
 U 1 1 57B9D3A1
 P 4300 2150
@@
 $EndComp
 $Comp
-L GND #PWR011
+L icu-rescue:GND #PWR011
 U 1 1 57CF1F5E
 P 2800 5150
@@
 $EndComp
 $Comp
-L IND_744045210 L201
+L icu-rescue:IND_744045210 L201
 U 1 1 58945E39
 P 6500 3850
@@
 $EndComp
 $Comp
-L DIODE_RS07J-GS18 D201
+L icu-rescue:DIODE_RS07J-GS18 D201
 U 1 1 5896E2A2
 P 1900 3850
@@
 $EndComp
 $Comp
-L T491D226K035AT C204
+L icu-rescue:T491D226K035AT C204
 U 1 1 597AF606
 P 6850 4050
@@
 $EndComp
 $Comp
-L REG_MCP1700 VR202
+L icu-rescue:REG_MCP1700 VR202
 U 1 1 597AF83E
 P 8000 3950
@@
 $EndComp
 $Comp
-L SCHOTTKY_DIODE_V40PW10C D203
+L icu-rescue:SCHOTTKY_DIODE_V40PW10C D203
 U 1 1 59B7B8B2
 P 2050 3250
@@
 $EndComp
 $Comp
-L SCHOTTKY_DIODE_V40PW10C D202
+L icu-rescue:SCHOTTKY_DIODE_V40PW10C D202
 U 1 1 59D9089A
 P 2050 2750
@@
 $EndComp
 $Comp
-L CAP_EEE-FK1H470P C202
+L icu-rescue:CAP_EEE-FK1H470P C202
 U 1 1 5A13B69C
 P 3800 4050
@@
 $EndComp
 $Comp
-L DIODE_TVS_TPSMD28A D205
+L icu-rescue:DIODE_TVS_TPSMD28A D205
 U 1 1 5A13BC8E
 P 2900 2950
@@
 $EndComp
 $Comp
-L GND #PWR012
+L icu-rescue:GND #PWR012
 U 1 1 5A13BD77
 P 2900 3150
