File: hw/pwr_supply_sheet.sch (KiCad schematic (older format))
At the start: 15 parts

Commit message: 3.0.0 hw and gerber created
Parts:
- removed C203: 10nF, kemet:0603, symbol 10nF
- removed VR202: REG_MCP1700, usevolt:SOT-23_3-PIN, symbol REG_MCP1700
- added C1: 100nF, kemet:0603, symbol kemet:100nF
- added VR1: REG_MCP1700, usevolt:SOT-23_3-PIN, symbol usevolt:REG_MCP1700
- C201, C205: symbol 100nF -> kemet:100nF
- C202: symbol CAP_EEE-FK1H470P -> usevolt:CAP_EEE-FK1H470P
- C204: symbol T491D226K035AT -> kemet:T491D226K035AT
- D201, D206: symbol DIODE_RS07J-GS18 -> usevolt:DIODE_RS07J-GS18
- D202, D203: symbol SCHOTTKY_DIODE_V40PW10C -> usevolt:SCHOTTKY_DIODE_V40PW10C
- D204: symbol DIODE_TVS_SMBJ33A-TRDO-214AA -> usevolt:DIODE_TVS_SMBJ33A-TRDO-214AA
- D205: symbol DIODE_TVS_TPSMD28A -> usevolt:DIODE_TVS_TPSMD28A
- F201: symbol FUSE_MC36211_350MA -> usevolt:FUSE_MC36211_350MA
- L201: symbol IND_744045210 -> usevolt:IND_744045210
- VR201: symbol LM2671SOIC8 -> usevolt:LM2671SOIC8
Connections:
- net +3V3: now also VR1.P$2 (VOUT)
- net +5V: now also VR1.P$3 (VIN)
- net GND: now also VR1.P$1 (GND)
- net at VR201.1 (CB): now also C1.2 (C2)
- net at D206.P$2 (N), L201.1, VR201.8 (VSW): now also C1.1 (C1)
Changed lines of the file:
@@
-EESchema Schematic File Version 2
-LIBS:kemet
-LIBS:usevolt
-LIBS:wurth_elektronik_LED
-LIBS:power
-LIBS:yageo
+EESchema Schematic File Version 4
 LIBS:icu-cache
 EELAYER 26 0
@@
 VIN
 $Comp
-L FUSE_MC36211_350MA F201
+L usevolt:FUSE_MC36211_350MA F201
 U 1 1 57B8204F
 P 2500 3850
@@
 $EndComp
 $Comp
-L DIODE_TVS_SMBJ33A-TRDO-214AA D204
+L usevolt:DIODE_TVS_SMBJ33A-TRDO-214AA D204
 U 1 1 57B820C1
 P 2800 4050
@@
 $EndComp
 $Comp
-L 100nF C201
+L kemet:100nF C201
 U 1 1 57B8217A
 P 3400 3950
@@
 $EndComp
 $Comp
-L LM2671SOIC8 VR?
+L usevolt:LM2671SOIC8 VR?
 U 1 1 57B82261
 P 4850 4150
@@
 $EndComp
 $Comp
-L 10nF C203
-U 1 1 57B822C5
-P 5800 3950
-F 0 "C203" H 5850 4149 45  0000 C CNN
-F 1 "10nF" H 5850 4065 45  0000 C CNN
-F 2 "kemet:0603" H 5830 4100 20  0001 C CNN
-F 3 "http://www.farnell.com/datasheets/2064086.pdf?_ga=1.250530118.1948984246.1460023966" H 5704 3959 60  0001 C CNN
-F 4 "1457729" H 6104 4359 60  0001 C CNN "1st Source Part Number"
-F 5 "C0603C103J3GACTU" H 5904 4159 60  0001 C CNN "Manufacturer Part Number"
-F 6 "Farnell" H 6004 4259 60  0001 C CNN "1st Source"
-F 7 "KEMET" H 5804 4059 60  0001 C CNN "Manufacturer"
-	1    5800 3950
-	1    0    0    -1
-$EndComp
-$Comp
-L DIODE_RS07J-GS18 D206
+L usevolt:DIODE_RS07J-GS18 D206
 U 1 1 57B82329
 P 6200 3950
@@
 $EndComp
 $Comp
-L 100nF C205
+L kemet:100nF C205
 U 1 1 57B82A3F
 P 8600 3950
@@
 $EndComp
 $Comp
-L +5V #PWR05
+L power:+5V #PWR05
 U 1 1 57B831F8
 P 6850 3600
@@
 $EndComp
 $Comp
-L +3V3 #PWR06
+L power:+3V3 #PWR06
 U 1 1 57B83259
 P 8600 3600
@@
 NoConn ~ 4550 4050
 $Comp
-L VDD #PWR07
+L power:VDD #PWR07
 U 1 1 57B9C56A
 P 3800 2100
@@
 $EndComp
 $Comp
-L PWR_FLAG #FLG08
+L power:PWR_FLAG #FLG08
 U 1 1 57B9C59C
 P 3800 2300
@@
 $EndComp
 $Comp
-L GND #PWR09
+L power:GND #PWR09
 U 1 1 57B9D351
 P 4300 2350
@@
 $EndComp
 $Comp
-L PWR_FLAG #FLG010
+L power:PWR_FLAG #FLG010
 U 1 1 57B9D3A1
 P 4300 2150
@@
 $EndComp
 $Comp
-L GND #PWR011
+L power:GND #PWR011
 U 1 1 57CF1F5E
 P 2800 5150
@@
 $EndComp
 $Comp
-L IND_744045210 L201
+L usevolt:IND_744045210 L201
 U 1 1 58945E39
 P 6500 3850
@@
 $EndComp
 $Comp
-L DIODE_RS07J-GS18 D201
+L usevolt:DIODE_RS07J-GS18 D201
 U 1 1 5896E2A2
 P 1900 3850
@@
 $EndComp
 $Comp
-L T491D226K035AT C204
+L kemet:T491D226K035AT C204
 U 1 1 597AF606
 P 6850 4050
@@
 $EndComp
 $Comp
-L REG_MCP1700 VR202
-U 1 1 597AF83E
-P 8000 3950
-F 0 "VR202" H 8000 4305 45  0000 C CNN
-F 1 "REG_MCP1700" H 8000 3950 45  0001 L BNN
-F 2 "usevolt:SOT-23_3-PIN" H 8030 4100 20  0001 C CNN
-F 3 "http://www.farnell.com/datasheets/1784514.pdf?_ga=1.221693144.1948984246.1460023966" H 7700 4270 60  0001 C CNN
-F 4 "1296592" H 8100 4670 60  0001 C CNN "1st Source Part Number"
-F 5 "Digi-Key" H 8200 4770 60  0001 C CNN "2nd Source"
-F 6 "Farnell" H 8000 4570 60  0001 C CNN "1st Source"
-F 7 "MCP1700T-3302E/TT" H 7900 4470 60  0001 C CNN "Manufacturer Part Number"
-F 8 "MCP1700T3302ETTCT-ND" H 8300 4870 60  0001 C CNN "2nd Source Part Number"
-F 9 "MICROCHIP" H 7800 4370 60  0001 C CNN "Manufacturer"
-	1    8000 3950
-	1    0    0    -1
-$EndComp
-$Comp
-L SCHOTTKY_DIODE_V40PW10C D203
+L usevolt:SCHOTTKY_DIODE_V40PW10C D203
 U 1 1 59B7B8B2
 P 2050 3250
@@
 $EndComp
 $Comp
-L SCHOTTKY_DIODE_V40PW10C D202
+L usevolt:SCHOTTKY_DIODE_V40PW10C D202
 U 1 1 59D9089A
 P 2050 2750
@@
 $EndComp
 $Comp
-L CAP_EEE-FK1H470P C202
+L usevolt:CAP_EEE-FK1H470P C202
 U 1 1 5A13B69C
 P 3800 4050
@@
 $EndComp
 $Comp
-L DIODE_TVS_TPSMD28A D205
+L usevolt:DIODE_TVS_TPSMD28A D205
 U 1 1 5A13BC8E
 P 2900 2950
@@
 $EndComp
 $Comp
-L GND #PWR012
+L power:GND #PWR012
 U 1 1 5A13BD77
 P 2900 3150
@@
 Connection ~ 3800 4950
 Wire Wire Line
-	2800 4150 2800 5150
+	2800 4150 2800 4950
 Connection ~ 3400 4950
 Connection ~ 2800 3850
@@
 	8600 3850 8400 3850
 Wire Wire Line
-	6700 3850 7600 3850
+	6700 3850 6850 3850
 Connection ~ 6850 3850
 Wire Wire Line
-	5550 3850 6300 3850
+	5550 3850 6000 3850
 Connection ~ 6200 3850
 Wire Wire Line
@@
 	5550 3750 6850 3750
 Wire Wire Line
-	6850 3600 6850 3850
+	6850 3600 6850 3750
 Connection ~ 6850 3750
 Wire Wire Line
-	1350 3850 1700 3850
+	1350 3850 1500 3850
 Wire Wire Line
 	3800 3700 4550 3700
@@
 Connection ~ 1500 3850
 Wire Wire Line
-	2700 3850 3800 3850
+	2700 3850 2800 3850
 Wire Wire Line
 	2000 3850 2300 3850
 Wire Wire Line
-	2700 4950 8600 4950
+	2700 4950 2800 4950
 Wire Wire Line
 	2750 3200 2450 3200
@@
 Connection ~ 1500 2750
 Wire Wire Line
-	2450 2700 3150 2700
+	2450 2700 2750 2700
 Wire Wire Line
 	2750 2700 2750 3200
@@
 	2900 3150 2900 3050
 Wire Wire Line
-	1500 3850 1500 2650
+	1500 3850 1500 3250
+Wire Wire Line
+	8000 4950 8600 4950
+Wire Wire Line
+	6850 4950 8000 4950
+Wire Wire Line
+	6200 4950 6850 4950
+Wire Wire Line
+	5550 4950 6200 4950
+Wire Wire Line
+	3800 4950 5550 4950
+Wire Wire Line
+	3400 4950 3800 4950
+Wire Wire Line
+	2800 3850 3400 3850
+Wire Wire Line
+	3400 3850 3800 3850
+Wire Wire Line
+	6850 3850 7600 3850
+Wire Wire Line
+	6200 3850 6300 3850
+Wire Wire Line
+	6000 3850 6200 3850
+Wire Wire Line
+	6850 3750 6850 3850
+Wire Wire Line
+	2800 4950 2800 5150
+Wire Wire Line
+	2800 4950 3400 4950
+Wire Wire Line
+	1500 3850 1700 3850
+Wire Wire Line
+	1500 3250 1500 3150
+Wire Wire Line
+	1500 3150 1500 2750
+Wire Wire Line
+	1500 2750 1500 2650
+Wire Wire Line
+	2750 2700 2900 2700
+Wire Wire Line
+	2900 2700 3150 2700
+$Comp
+L usevolt:REG_MCP1700 VR1
+U 1 1 5BB6A08A
+P 8000 3950
+F 0 "VR1" H 8000 4305 45  0000 C CNN
+F 1 "REG_MCP1700" H 8000 3950 45  0001 L BNN
+F 2 "usevolt:SOT-23_3-PIN" H 8030 4100 20  0001 C CNN
+F 3 "http://www.farnell.com/datasheets/1784514.pdf?_ga=1.221693144.1948984246.1460023966" H 7700 4270 60  0001 C CNN
+F 4 "1296592" H 8100 4670 60  0001 C CNN "1st Source Part Number"
+F 5 "Digi-Key" H 8200 4770 60  0001 C CNN "2nd Source"
+F 6 "Farnell" H 8000 4570 60  0001 C CNN "1st Source"
+F 7 "MCP1700T-3302E/TT" H 7900 4470 60  0001 C CNN "Manufacturer Part Number"
+F 8 "MCP1700T3302ETTCT-ND" H 8300 4870 60  0001 C CNN "2nd Source Part Number"
+F 9 "MICROCHIP" H 7800 4370 60  0001 C CNN "Manufacturer"
+	1    8000 3950
+	1    0    0    -1
+$EndComp
+$Comp
+L kemet:100nF C1
+U 1 1 5BB73960
+P 5900 3950
+F 0 "C1" V 5908 4023 45  0000 L CNN
+F 1 "100nF" V 5992 4023 45  0000 L CNN
+F 2 "kemet:0603" H 5930 4100 20  0001 C CNN
+F 3 "http://www.farnell.com/datasheets/2062872.pdf?_ga=1.250530118.1948984246.1460023966" H 5804 3959 60  0001 C CNN
+F 4 "1288255" H 6204 4359 60  0001 C CNN "1st Source Part Number"
+F 5 "C0603C104K5RACTU" H 6004 4159 60  0001 C CNN "Manufacturer Part Number"
+F 6 "Farnell" H 6104 4259 60  0001 C CNN "1st Source"
+F 7 "KEMET" H 5904 4059 60  0001 C CNN "Manufacturer"
+	1    5900 3950
+	-1   0    0    1
+$EndComp
 $EndSCHEMATC
