File: hw/lpc1549.sch (KiCad schematic (older format))
At the start: 18 parts, among them J1001 ARM_JTAG_SWD_HEADER_10_PINSMD, U1001 MCP2551_SOIC8, U1002 LPC1549JBD64, X1001 XTAL_7A-12.000MAAJ-T

Commit message: hw 1.0 ready to order
Parts:
- added R907: 1K, yageo:0603, symbol 1K
Connections:
- net AIN1: now also U1002.P$9 (PIO0_5/ADC0_3); no longer U1002.P$8 (PIO0_4/ADC0_4)
- net AIN2: now also U1002.P$8 (PIO0_4/ADC0_4); no longer U1002.P$9 (PIO0_5/ADC0_3)
- net AIN3: now also U1002.P$4 (PIO1_0/ADC0_8); no longer U1002.P$11 (PIO0_7/ADC0_1)
- net OUT1_1: now also U1002.P$58 (PIO0_24/SCT0_OUT6); no longer U1002.P$5 (PIO0_1/ADC0_7/SCT0_OUT4)
- net OUT1_2: now also U1002.P$53 (PIO1_8/ACMP3_I3/SCT3_OUT4); no longer U1002.P$6 (PIO0_2/ADC0_6/SCT1_OUT3)
- net OUT1_SENSE: now also U1002.P$34 (PIO1_5/ADC1_11); no longer U1002.P$3 (PIO0_31/ADC0_9)
- net OUT2_1: now also U1002.P$64 (PIO0_29/ACMP2_I3/SCT2_OUT4); no longer U1002.P$7 (PIO0_3/ADC0_5/SCT1_OUT4)
- net OUT2_2: now also U1002.P$61 (PIO0_26/ACMP0_I3/SCT3_OUT3); no longer U1002.P$2 (PIO0_0/ADC0_10/SCT0_OUT3)
- net OUT2_SENSE: now also U1002.P$33 (PIO1_4/ADC1_10); no longer U1002.P$1 (PIO0_30/ADC0_11)
- net OUT3_1: now also U1002.P$5 (PIO0_1/ADC0_7/SCT0_OUT4); no longer U1002.P$10 (PIO0_6/ADC0_2/SCT2_OUT3)
- net OUT3_2: now also U1002.P$2 (PIO0_0/ADC0_10/SCT0_OUT3); no longer U1002.P$30 (PIO0_14/ADC1_7/SCT1_OUT5)
- net OUT3_SENSE: now also U1002.P$31 (PIO0_15/ADC1_8); no longer U1002.P$4 (PIO1_0/ADC0_8)
- net OUT4_1: now also U1002.P$7 (PIO0_3/ADC0_5/SCT1_OUT4); no longer U1002.P$53 (PIO1_8/ACMP3_I3/SCT3_OUT4)
- net OUT4_2: now also U1002.P$6 (PIO0_2/ADC0_6/SCT1_OUT3); no longer U1002.P$58 (PIO0_24/SCT0_OUT6)
- net OUT4_SENSE: now also U1002.P$32 (PIO0_16/ADC1_9); no longer U1002.P$29 (PIO0_13/ADC1_6)
- net OUT5_1: now also U1002.P$30 (PIO0_14/ADC1_7/SCT1_OUT5); no longer U1002.P$61 (PIO0_26/ACMP0_I3/SCT3_OUT3)
- net OUT5_2: now also U1002.P$10 (PIO0_6/ADC0_2/SCT2_OUT3); no longer U1002.P$64 (PIO0_29/ACMP2_I3/SCT2_OUT4)
- net OUT6_1: now also U1002.P$19 (PIO0_10/ADC1_2); no longer U1002.P$17 (PIO0_18/SCT0_OUT5)
- net OUT6_2: now also U1002.P$24 (PIO0_12/DAC_OUT); no longer U1002.P$19 (PIO0_10/ADC1_2)
- net OUT6_SENSE: now also U1002.P$11 (PIO0_7/ADC0_1); no longer U1002.P$31 (PIO0_15/ADC1_8)
- net OUT7_1: now also U1002.P$17 (PIO0_18/SCT0_OUT5); no longer U1002.P$24 (PIO0_12/DAC_OUT)
- net OUT7_2: now also U1002.P$16 (PIO0_9/ADC1_1/TDI); no longer U1002.P$62 (PIO0_27/ACMP_I1)
- net OUT7_SENSE: now also U1002.P$12 (PIO0_8/ADC0_0/TDO); no longer U1002.P$32 (PIO0_16/ADC1_9)
- net at R904.1 (R1): now also U1002.P$1 (PIO0_30/ADC0_11); no longer U1002.P$15 (PIO1_1/ADC1_0)
- net at R905.1 (R1): now also U1002.P$63 (PIO0_28/ACMP1_I3); no longer U1002.P$16 (PIO0_9/ADC1_1/TDI)
- net at U1002.P$23 (PIO0_11/ADC1_3): no longer R906.1 (R1)
- net at U1002.P$51 (PIO1_7/ADCMP3_I4): now also R907.2 (R2)
- new net: R906.1 (R1), U1002.P$62 (PIO0_27/ACMP_I1)
- new net AIN4: U1002.P$3 (PIO0_31/ADC0_9)
- new net DIN4: R907.1 (R1)
Other:
- moved on the sheet: R904, R905, R906
Changed lines of the file:
@@
 $Descr A4 11693 8268
 encoding utf-8
-Sheet 9 13
+Sheet 9 14
 Title ""
 Date ""
@@
 $EndComp
 $Comp
-L +3V3 #PWR903
+L +3V3 #PWR037
 U 1 1 57E689A3
 P 3600 3950
-F 0 "#PWR903" H 3600 3800 50  0001 C CNN
+F 0 "#PWR037" H 3600 3800 50  0001 C CNN
 F 1 "+3V3" H 3615 4123 50  0000 C CNN
 F 2 "" H 3600 3950 50  0000 C CNN
@@
 $EndComp
 $Comp
-L GND #PWR904
+L GND #PWR038
 U 1 1 57E689C9
 P 3600 4550
-F 0 "#PWR904" H 3600 4300 50  0001 C CNN
+F 0 "#PWR038" H 3600 4300 50  0001 C CNN
 F 1 "GND" H 3605 4377 50  0000 C CNN
 F 2 "" H 3600 4550 50  0000 C CNN
@@
 $EndComp
 $Comp
-L GND #PWR906
+L GND #PWR039
 U 1 1 57E697A1
 P 8000 3100
-F 0 "#PWR906" H 8000 2850 50  0001 C CNN
+F 0 "#PWR039" H 8000 2850 50  0001 C CNN
 F 1 "GND" H 8005 2927 50  0000 C CNN
 F 2 "" H 8000 3100 50  0000 C CNN
@@
 $EndComp
 $Comp
-L GND #PWR905
+L GND #PWR040
 U 1 1 57E69A8B
 P 7300 3350
-F 0 "#PWR905" H 7300 3100 50  0001 C CNN
+F 0 "#PWR040" H 7300 3100 50  0001 C CNN
 F 1 "GND" H 7305 3177 50  0000 C CNN
 F 2 "" H 7300 3350 50  0000 C CNN
@@
 $EndComp
 $Comp
-L GND #PWR907
+L GND #PWR041
 U 1 1 5891FBFB
 P 9700 4500
-F 0 "#PWR907" H 9700 4250 50  0001 C CNN
+F 0 "#PWR041" H 9700 4250 50  0001 C CNN
 F 1 "GND" H 9705 4327 50  0000 C CNN
 F 2 "" H 9700 4500 50  0000 C CNN
@@
 $EndComp
 $Comp
-L +3V3 #PWR908
+L +3V3 #PWR042
 U 1 1 5891FCDE
 P 9750 3450
-F 0 "#PWR908" H 9750 3300 50  0001 C CNN
+F 0 "#PWR042" H 9750 3300 50  0001 C CNN
 F 1 "+3V3" H 9765 3623 50  0000 C CNN
 F 2 "" H 9750 3450 50  0000 C CNN
@@
 Connection ~ 9750 3450
 $Comp
-L +5V #PWR901
+L +5V #PWR043
 U 1 1 58C01582
 P 2800 2750
-F 0 "#PWR901" H 2800 2600 50  0001 C CNN
+F 0 "#PWR043" H 2800 2600 50  0001 C CNN
 F 1 "+5V" H 2815 2923 50  0000 C CNN
 F 2 "" H 2800 2750 50  0000 C CNN
@@
 $EndComp
 $Comp
-L GND #PWR902
+L GND #PWR044
 U 1 1 58C01588
 P 2800 3300
-F 0 "#PWR902" H 2800 3050 50  0001 C CNN
+F 0 "#PWR044" H 2800 3050 50  0001 C CNN
 F 1 "GND" H 2805 3127 50  0000 C CNN
 F 2 "" H 2800 3300 50  0000 C CNN
@@
 $EndComp
 Wire Wire Line
+	7000 4950 7300 4950
+Wire Wire Line
+	7000 4850 7300 4850
+Wire Wire Line
+	7000 5750 7300 5750
+Text HLabel 7300 4950 2    60   Output ~ 0
+OUT1_1
+Text HLabel 7300 4850 2    60   Output ~ 0
+OUT1_2
+Text HLabel 7300 5750 2    60   Output ~ 0
+OUT2_1
+Wire Wire Line
+	7000 5450 7300 5450
+Text HLabel 7300 5450 2    60   Output ~ 0
+OUT2_2
+Wire Wire Line
 	5200 2550 4900 2550
-Wire Wire Line
-	5200 2650 4900 2650
-Wire Wire Line
-	5200 2750 4900 2750
 Text HLabel 4900 2550 0    60   Output ~ 0
-OUT1_1
-Text HLabel 4900 2650 0    60   Output ~ 0
-OUT1_2
-Text HLabel 4900 2750 0    60   Output ~ 0
-OUT2_1
+OUT3_1
 Wire Wire Line
 	5200 2250 4900 2250
 Text HLabel 4900 2250 0    60   Output ~ 0
-OUT2_2
+OUT3_2
+Wire Wire Line
+	5200 2750 4900 2750
+Text HLabel 4900 2750 0    60   Output ~ 0
+OUT4_1
+Wire Wire Line
+	5200 2650 4900 2650
+Text HLabel 4900 2650 0    60   Output ~ 0
+OUT4_2
+Wire Wire Line
+	7000 2150 7300 2150
+Text HLabel 7300 2150 2    60   Output ~ 0
+OUT5_1
 Wire Wire Line
 	5200 3050 4900 3050
 Text HLabel 4900 3050 0    60   Output ~ 0
-OUT3_1
-Wire Wire Line
-	7000 2150 7300 2150
-Text HLabel 7300 2150 2    60   Output ~ 0
-OUT3_2
-Wire Wire Line
-	7000 4850 7300 4850
-Text HLabel 7300 4850 2    60   Output ~ 0
-OUT4_1
-Wire Wire Line
-	7000 4950 7300 4950
-Text HLabel 7300 4950 2    60   Output ~ 0
-OUT4_2
-Wire Wire Line
-	7000 5450 7300 5450
-Text HLabel 7300 5450 2    60   Output ~ 0
-OUT5_1
-Wire Wire Line
-	7000 5750 7300 5750
-Text HLabel 7300 5750 2    60   Output ~ 0
 OUT5_2
+Wire Wire Line
+	5200 5350 4900 5350
+Text HLabel 4900 5350 0    60   Output ~ 0
+OUT6_1
+Wire Wire Line
+	5200 5650 4900 5650
+Text HLabel 4900 5650 0    60   Output ~ 0
+OUT6_2
 Wire Wire Line
 	5200 5250 4900 5250
 Text HLabel 4900 5250 0    60   Output ~ 0
-OUT6_1
-Wire Wire Line
-	5200 5350 4900 5350
-Text HLabel 4900 5350 0    60   Output ~ 0
-OUT6_2
-Wire Wire Line
-	5200 5650 4900 5650
-Text HLabel 4900 5650 0    60   Output ~ 0
 OUT7_1
 Wire Wire Line
-	7000 5550 7300 5550
-Text HLabel 7300 5550 2    60   Output ~ 0
+	5200 5150 4900 5150
+Text HLabel 4900 5150 0    60   Output ~ 0
 OUT7_2
 Wire Wire Line
-	5200 2150 4900 2150
-Text HLabel 4900 2150 0    60   Input ~ 0
+	7000 2550 7300 2550
+Text HLabel 7300 2550 2    60   Input ~ 0
 OUT2_SENSE
 Wire Wire Line
-	5200 2350 4900 2350
-Text HLabel 4900 2350 0    60   Input ~ 0
+	7000 2650 7300 2650
+Text HLabel 7300 2650 2    60   Input ~ 0
 OUT1_SENSE
 Wire Wire Line
-	5200 2450 4900 2450
-Text HLabel 4900 2450 0    60   Input ~ 0
+	7000 2350 7300 2350
+Text HLabel 7300 2350 2    60   Input ~ 0
 OUT3_SENSE
 Wire Wire Line
-	7000 2050 7300 2050
-Text HLabel 7300 2050 2    60   Input ~ 0
+	7000 2450 7300 2450
+Text HLabel 7300 2450 2    60   Input ~ 0
 OUT4_SENSE
 Wire Wire Line
@@
 OUT5_SENSE
 Wire Wire Line
-	7000 2350 7300 2350
-Text HLabel 7300 2350 2    60   Input ~ 0
+	5200 3150 4900 3150
+Text HLabel 4900 3150 0    60   Input ~ 0
 OUT6_SENSE
 Wire Wire Line
-	7000 2450 7300 2450
-Text HLabel 7300 2450 2    60   Input ~ 0
+	5200 3250 4900 3250
+Text HLabel 4900 3250 0    60   Input ~ 0
 OUT7_SENSE
 Wire Wire Line
-	5200 5050 4650 5050
-Wire Wire Line
-	5200 5150 4650 5150
-Text HLabel 4250 5050 0    60   Input ~ 0
+	5200 2150 4650 2150
+Wire Wire Line
+	7000 5650 7550 5650
+Text HLabel 4250 2150 0    60   Input ~ 0
 DIN1
-Text HLabel 4250 5150 0    60   Input ~ 0
+Text HLabel 7950 5650 2    60   Input ~ 0
 DIN2
 Wire Wire Line
-	5200 5550 4650 5550
-Text HLabel 4250 5550 0    60   Input ~ 0
+	7000 5550 7550 5550
+Text HLabel 7950 5550 2    60   Input ~ 0
 DIN3
 $Comp
 L 1K R904
 U 1 1 5A7DF40A
-P 4450 5050
-F 0 "R904" H 4500 5234 45  0000 C CNN
-F 1 "1K" H 4500 5150 45  0000 C CNN
-F 2 "yageo:0603" H 4480 5200 20  0001 C CNN
-F 3 "" H 4419 5089 60  0001 C CNN
-F 4 "" H 4819 5489 60  0001 C CNN "1st Source Part Number"
-F 5 "Digikey" H 4719 5389 60  0001 C CNN "1st Source"
-F 6 "RC0603FR-071KL" H 4619 5289 60  0001 C CNN "Manufacturer Part Number"
-F 7 "YAGEO" H 4519 5189 60  0001 C CNN "Manufacturer"
-	1    4450 5050
+P 4450 2150
+F 0 "R904" H 4500 2334 45  0000 C CNN
+F 1 "1K" H 4500 2250 45  0000 C CNN
+F 2 "yageo:0603" H 4480 2300 20  0001 C CNN
+F 3 "" H 4419 2189 60  0001 C CNN
+F 4 "" H 4819 2589 60  0001 C CNN "1st Source Part Number"
+F 5 "Digikey" H 4719 2489 60  0001 C CNN "1st Source"
+F 6 "RC0603FR-071KL" H 4619 2389 60  0001 C CNN "Manufacturer Part Number"
+F 7 "YAGEO" H 4519 2289 60  0001 C CNN "Manufacturer"
+	1    4450 2150
 	1    0    0    -1
 $EndComp
@@
 L 1K R905
 U 1 1 5A7DF46E
-P 4450 5150
-F 0 "R905" H 4500 5334 45  0000 C CNN
-F 1 "1K" H 4500 5250 45  0000 C CNN
-F 2 "yageo:0603" H 4480 5300 20  0001 C CNN
-F 3 "" H 4419 5189 60  0001 C CNN
-F 4 "" H 4819 5589 60  0001 C CNN "1st Source Part Number"
-F 5 "Digikey" H 4719 5489 60  0001 C CNN "1st Source"
-F 6 "RC0603FR-071KL" H 4619 5389 60  0001 C CNN "Manufacturer Part Number"
-F 7 "YAGEO" H 4519 5289 60  0001 C CNN "Manufacturer"
-	1    4450 5150
-	1    0    0    -1
+P 7750 5650
+F 0 "R905" H 7800 5834 45  0000 C CNN
+F 1 "1K" H 7800 5750 45  0000 C CNN
+F 2 "yageo:0603" H 7780 5800 20  0001 C CNN
+F 3 "" H 7719 5689 60  0001 C CNN
+F 4 "" H 8119 6089 60  0001 C CNN "1st Source Part Number"
+F 5 "Digikey" H 8019 5989 60  0001 C CNN "1st Source"
+F 6 "RC0603FR-071KL" H 7919 5889 60  0001 C CNN "Manufacturer Part Number"
+F 7 "YAGEO" H 7819 5789 60  0001 C CNN "Manufacturer"
+	1    7750 5650
+	-1   0    0    -1
 $EndComp
 $Comp
 L 1K R906
 U 1 1 5A7DF4BB
-P 4450 5550
-F 0 "R906" H 4500 5734 45  0000 C CNN
-F 1 "1K" H 4500 5650 45  0000 C CNN
-F 2 "yageo:0603" H 4480 5700 20  0001 C CNN
-F 3 "" H 4419 5589 60  0001 C CNN
-F 4 "" H 4819 5989 60  0001 C CNN "1st Source Part Number"
-F 5 "Digikey" H 4719 5889 60  0001 C CNN "1st Source"
-F 6 "RC0603FR-071KL" H 4619 5789 60  0001 C CNN "Manufacturer Part Number"
-F 7 "YAGEO" H 4519 5689 60  0001 C CNN "Manufacturer"
-	1    4450 5550
-	1    0    0    -1
-$EndComp
-Wire Wire Line
-	4350 5150 4250 5150
-Wire Wire Line
-	4250 5050 4350 5050
-Wire Wire Line
-	4350 5550 4250 5550
+P 7750 5550
+F 0 "R906" H 7800 5734 45  0000 C CNN
+F 1 "1K" H 7800 5650 45  0000 C CNN
+F 2 "yageo:0603" H 7780 5700 20  0001 C CNN
+F 3 "" H 7719 5589 60  0001 C CNN
+F 4 "" H 8119 5989 60  0001 C CNN "1st Source Part Number"
+F 5 "Digikey" H 8019 5889 60  0001 C CNN "1st Source"
+F 6 "RC0603FR-071KL" H 7919 5789 60  0001 C CNN "Manufacturer Part Number"
+F 7 "YAGEO" H 7819 5689 60  0001 C CNN "Manufacturer"
+	1    7750 5550
+	-1   0    0    -1
+$EndComp
+Wire Wire Line
+	7850 5650 7950 5650
+Wire Wire Line
+	4250 2150 4350 2150
+Wire Wire Line
+	7850 5550 7950 5550
+Wire Wire Line
+	5200 2950 4900 2950
+Text HLabel 4900 2950 0    60   Input ~ 0
+AIN1
 Wire Wire Line
 	5200 2850 4900 2850
 Text HLabel 4900 2850 0    60   Input ~ 0
-AIN1
-Wire Wire Line
-	5200 2950 4900 2950
-Text HLabel 4900 2950 0    60   Input ~ 0
 AIN2
 Wire Wire Line
-	5200 3150 4900 3150
-Text HLabel 4900 3150 0    60   Input ~ 0
+	5200 2450 4900 2450
+Text HLabel 4900 2450 0    60   Input ~ 0
 AIN3
+Wire Wire Line
+	5200 2350 4900 2350
+Text HLabel 4900 2350 0    60   Input ~ 0
+AIN4
+Text HLabel 8300 4750 2    60   Input ~ 0
+DIN4
+$Comp
+L 1K R907
+U 1 1 5A8C941E
+P 8050 4750
+F 0 "R907" H 8100 4934 45  0000 C CNN
+F 1 "1K" H 8100 4850 45  0000 C CNN
+F 2 "yageo:0603" H 8080 4900 20  0001 C CNN
+F 3 "" H 8019 4789 60  0001 C CNN
+F 4 "" H 8419 5189 60  0001 C CNN "1st Source Part Number"
+F 5 "Digikey" H 8319 5089 60  0001 C CNN "1st Source"
+F 6 "RC0603FR-071KL" H 8219 4989 60  0001 C CNN "Manufacturer Part Number"
+F 7 "YAGEO" H 8119 4889 60  0001 C CNN "Manufacturer"
+	1    8050 4750
+	1    0    0    -1
+$EndComp
+Wire Wire Line
+	7950 4750 7000 4750
+Wire Wire Line
+	8250 4750 8300 4750
 $EndSCHEMATC

Commit message: 3.0.0 hw and gerber created
Parts:
- C1001, C1002, C1003, C1004, C1005, C1006, C1007: symbol 100nF -> kemet:100nF
- C1008, C1009: symbol 18pF -> kemet:18pF
- J1001: symbol ARM_JTAG_SWD_HEADER_10_PINSMD -> usevolt:ARM_JTAG_SWD_HEADER_10_PINSMD
- R1001, R1002: symbol 10K -> yageo:10K
- R904, R905, R906, R907: symbol 1K -> yageo:1K
- U1001: symbol MCP2551_SOIC8 -> usevolt:MCP2551_SOIC8
- U1002: symbol LPC1549JBD64 -> usevolt:LPC1549JBD64
- X1001: symbol XTAL_7A-12.000MAAJ-T -> usevolt:XTAL_7A-12.000MAAJ-T
Changed lines of the file:
@@
-EESchema Schematic File Version 2
-LIBS:kemet
-LIBS:usevolt
-LIBS:wurth_elektronik_LED
-LIBS:power
-LIBS:yageo
+EESchema Schematic File Version 4
 LIBS:icu-cache
 EELAYER 26 0
@@
 $EndDescr
 $Comp
-L 100nF C1007
+L kemet:100nF C1007
 U 1 1 57E685B4
 P 5000 4200
@@
 $EndComp
 $Comp
-L 100nF C1006
+L kemet:100nF C1006
 U 1 1 57E68621
 P 4650 4200
@@
 $EndComp
 $Comp
-L 100nF C1005
+L kemet:100nF C1005
 U 1 1 57E68672
 P 4300 4200
@@
 $EndComp
 $Comp
-L 100nF C1004
+L kemet:100nF C1004
 U 1 1 57E686C7
 P 3950 4200
@@
 $EndComp
 $Comp
-L 100nF C1003
+L kemet:100nF C1003
 U 1 1 57E6871C
 P 3600 4200
@@
 $EndComp
 $Comp
-L +3V3 #PWR037
+L power:+3V3 #PWR037
 U 1 1 57E689A3
 P 3600 3950
@@
 $EndComp
 $Comp
-L GND #PWR038
+L power:GND #PWR038
 U 1 1 57E689C9
 P 3600 4550
@@
 $EndComp
 $Comp
-L XTAL_7A-12.000MAAJ-T X1001
+L usevolt:XTAL_7A-12.000MAAJ-T X1001
 U 1 1 57E6956F
 P 7250 2950
@@
 $EndComp
 $Comp
-L 18pF C1008
+L kemet:18pF C1008
 U 1 1 57E695FA
 P 7550 2750
@@
 $EndComp
 $Comp
-L 18pF C1009
+L kemet:18pF C1009
 U 1 1 57E69648
 P 7550 3050
@@
 $EndComp
 $Comp
-L GND #PWR039
+L power:GND #PWR039
 U 1 1 57E697A1
 P 8000 3100
@@
 $EndComp
 $Comp
-L GND #PWR040
+L power:GND #PWR040
 U 1 1 57E69A8B
 P 7300 3350
@@
 $EndComp
 $Comp
-L GND #PWR041
+L power:GND #PWR041
 U 1 1 5891FBFB
 P 9700 4500
@@
 $EndComp
 $Comp
-L +3V3 #PWR042
+L power:+3V3 #PWR042
 U 1 1 5891FCDE
 P 9750 3450
@@
 Connection ~ 9750 3450
 $Comp
-L +5V #PWR043
+L power:+5V #PWR043
 U 1 1 58C01582
 P 2800 2750
@@
 $EndComp
 $Comp
-L GND #PWR044
+L power:GND #PWR044
 U 1 1 58C01588
 P 2800 3300
@@
 $EndComp
 $Comp
-L 100nF C?
+L kemet:100nF C?
 U 1 1 58C01592
 P 2900 2950
@@
 	1800 2950 1950 2950
 $Comp
-L 100nF C1002
+L kemet:100nF C1002
 U 1 1 58D0A5A6
 P 3250 4200
@@
 Connection ~ 5000 4400
 $Comp
-L LPC1549JBD64 U1002
+L usevolt:LPC1549JBD64 U1002
 U 1 1 59C4D0FB
 P 5700 2750
@@
 	9150 3650 9150 3950
 $Comp
-L MCP2551_SOIC8 U1001
+L usevolt:MCP2551_SOIC8 U1001
 U 1 1 5A102A85
 P 2350 2950
@@
 	2650 3050 2800 3050
 $Comp
-L 10K R1002
+L yageo:10K R1002
 U 1 1 5A533409
 P 9500 3600
@@
 $EndComp
 $Comp
-L 10K R1001
+L yageo:10K R1001
 U 1 1 5A533486
 P 9250 3550
@@
 $EndComp
 $Comp
-L ARM_JTAG_SWD_HEADER_10_PINSMD J1001
+L usevolt:ARM_JTAG_SWD_HEADER_10_PINSMD J1001
 U 1 1 5A79DD45
 P 9950 3950
@@
 DIN3
 $Comp
-L 1K R904
+L yageo:1K R904
 U 1 1 5A7DF40A
 P 4450 2150
@@
 $EndComp
 $Comp
-L 1K R905
+L yageo:1K R905
 U 1 1 5A7DF46E
 P 7750 5650
@@
 $EndComp
 $Comp
-L 1K R906
+L yageo:1K R906
 U 1 1 5A7DF4BB
 P 7750 5550
@@
 DIN4
 $Comp
-L 1K R907
+L yageo:1K R907
 U 1 1 5A8C941E
 P 8050 4750

Commit message: 3.3 pcb created
Connections:
- net AIN3: no longer names the net of U1002.P$4 (PIO1_0/ADC0_8)
- net AIN4: no longer names the net of U1002.P$3 (PIO0_31/ADC0_9)
Changed lines of the file:
@@
 $Descr A4 11693 8268
 encoding utf-8
-Sheet 9 14
+Sheet 9 12
 Title ""
 Date ""
@@
 RESET
 Wire Wire Line
-	5000 4400 5000 4900
-Wire Wire Line
-	5000 4500 5200 4500
+	5000 4400 5000 4500
+Wire Wire Line
+	5000 4500 5100 4500
 Wire Wire Line
 	5200 4400 5100 4400
@@
 Connection ~ 5100 4500
 Wire Wire Line
-	3250 4100 5200 4100
+	3250 4100 3600 4100
 Connection ~ 5000 4100
 Connection ~ 4650 4100
@@
 Connection ~ 3950 4100
 Wire Wire Line
-	3250 4400 5000 4400
+	3250 4400 3600 4400
 Connection ~ 3950 4400
 Connection ~ 4300 4400
@@
 Connection ~ 5000 3550
 Wire Wire Line
-	5000 3450 5000 4100
-Wire Wire Line
-	7100 3050 7450 3050
+	5000 3450 5000 3550
+Wire Wire Line
+	7100 3050 7250 3050
 Wire Wire Line
 	7100 3050 7100 2950
@@
 	7100 2850 7100 2750
 Wire Wire Line
-	7100 2750 7450 2750
+	7100 2750 7250 2750
 Connection ~ 7250 2750
 Wire Wire Line
 	7750 2750 8000 2750
 Wire Wire Line
-	8000 2750 8000 3100
+	8000 2750 8000 3050
 Wire Wire Line
 	8000 3050 7750 3050
@@
 	7600 5150 7000 5150
 Wire Wire Line
-	9150 3950 9850 3950
-Wire Wire Line
-	7000 3750 9850 3750
-Wire Wire Line
-	9700 3850 9700 4500
+	9150 3950 9500 3950
+Wire Wire Line
+	7000 3750 9250 3750
+Wire Wire Line
+	9700 3850 9700 4050
 Wire Wire Line
 	9700 4050 9850 4050
@@
 Connection ~ 9500 3950
 Wire Wire Line
-	9250 3450 9750 3450
+	9250 3450 9500 3450
 Wire Wire Line
 	9500 3500 9500 3450
@@
 $EndComp
 Wire Wire Line
-	2650 2850 2900 2850
+	2650 2850 2800 2850
 Wire Wire Line
 	2800 2850 2800 2750
 Wire Wire Line
-	2650 3150 2900 3150
-Wire Wire Line
-	2800 3050 2800 3300
+	2650 3150 2800 3150
+Wire Wire Line
+	2800 3050 2800 3150
 Connection ~ 2800 3150
 Connection ~ 2800 2850
@@
 Text HLabel 4900 2850 0    60   Input ~ 0
 AIN2
-Wire Wire Line
-	5200 2450 4900 2450
-Text HLabel 4900 2450 0    60   Input ~ 0
-AIN3
-Wire Wire Line
-	5200 2350 4900 2350
-Text HLabel 4900 2350 0    60   Input ~ 0
-AIN4
 Text HLabel 8300 4750 2    60   Input ~ 0
 DIN4
@@
 Wire Wire Line
 	8250 4750 8300 4750
+Wire Wire Line
+	5100 4500 5200 4500
+Wire Wire Line
+	5000 4100 5200 4100
+Wire Wire Line
+	4650 4100 5000 4100
+Wire Wire Line
+	4300 4100 4650 4100
+Wire Wire Line
+	3950 4100 4300 4100
+Wire Wire Line
+	3950 4400 4300 4400
+Wire Wire Line
+	4300 4400 4650 4400
+Wire Wire Line
+	4650 4400 5000 4400
+Wire Wire Line
+	5000 4500 5000 4600
+Wire Wire Line
+	5000 4600 5000 4700
+Wire Wire Line
+	5000 4700 5000 4800
+Wire Wire Line
+	5000 4800 5000 4900
+Wire Wire Line
+	5000 4000 5000 4100
+Wire Wire Line
+	5000 3900 5000 4000
+Wire Wire Line
+	5000 3800 5000 3900
+Wire Wire Line
+	5000 3700 5000 3800
+Wire Wire Line
+	5000 3550 5000 3700
+Wire Wire Line
+	7250 3050 7450 3050
+Wire Wire Line
+	7250 2750 7450 2750
+Wire Wire Line
+	8000 3050 8000 3100
+Wire Wire Line
+	9700 4050 9700 4500
+Wire Wire Line
+	9250 3750 9850 3750
+Wire Wire Line
+	9500 3950 9850 3950
+Wire Wire Line
+	9500 3450 9750 3450
+Wire Wire Line
+	2800 3150 2900 3150
+Wire Wire Line
+	2800 3150 2800 3300
+Wire Wire Line
+	2800 2850 2900 2850
+Wire Wire Line
+	3600 4400 3950 4400
+Wire Wire Line
+	3600 4100 3950 4100
 $EndSCHEMATC
