File: hw/vnd5050.sch (KiCad schematic (older format))
At the start: 8 parts, among them U301 VND5050AJTR-E

Commit message: CM_6.2.1 delivered, first customer machine with CCU, HCU & ICU
Parts:
- removed D801: ZENER_MM3Z3V6T1G, usevolt:SOD-323, symbol usevolt:ZENER_MM3Z3V6T1G
- removed R603: 1K, yageo:0603, symbol yageo:1K
- added D301: DIODE_RS07J-GS18, usevolt:DO219AB, symbol DIODE_RS07J-GS18
- added R303: 390, yageo:0603, symbol 390
- C301: symbol icu-rescue:4.7uF -> 4.7uF
- D302, D303: symbol icu-rescue:DIODE_RS07J-GS18 -> DIODE_RS07J-GS18
- R301, R302: symbol icu-rescue:1K -> 1K
- U301: symbol icu-rescue:VND5050AJTR-E -> VND5050AJTR-E
Connections:
- net GND: now also R303.2 (R2)
- net SENSE: now also D301.P$1 (P), R303.1 (R1)
- new net +3V3: D301.P$2 (N)
Changed lines of the file:
@@
-EESchema Schematic File Version 4
+EESchema Schematic File Version 2
+LIBS:kemet
+LIBS:usevolt
+LIBS:wurth_elektronik_LED
+LIBS:power
+LIBS:yageo
 LIBS:icu-cache
 EELAYER 26 0
@@
 $Descr A4 11693 8268
 encoding utf-8
-Sheet 8 13
+Sheet 4 14
 Title ""
 Date ""
@@
 SENSE
 $Comp
-L icu-rescue:VND5050AJTR-E U301
+L VND5050AJTR-E U301
 U 1 1 59D8088A
 P 4600 4000
@@
 $EndComp
 $Comp
-L icu-rescue:VDD #PWR045
+L VDD #PWR045
 U 1 1 59D808C7
 P 5250 3650
@@
 $EndComp
 $Comp
-L icu-rescue:GND #PWR046
+L GND #PWR046
 U 1 1 59D86DC2
 P 2950 4450
@@
 $EndComp
 $Comp
-L icu-rescue:1K R?
+L 390 R?
+U 1 1 59D88845
+P 3150 3550
+AR Path="/5A015FC0/59D88845" Ref="R?"  Part="1"
+AR Path="/5A02A41F/59D88845" Ref="R?"  Part="1"
+AR Path="/5A12B58E/59D88845" Ref="R?"  Part="1"
+AR Path="/5A7B157A/59D88845" Ref="R303"  Part="1"
+AR Path="/5A7B341B/59D88845" Ref="R503"  Part="1"
+AR Path="/5A7B2C1B/59D88845" Ref="R403"  Part="1"
+AR Path="/5A7B3FAD/59D88845" Ref="R603"  Part="1"
+AR Path="/5A7B4C13/59D88845" Ref="R703"  Part="1"
+AR Path="/5A7B577E/59D88845" Ref="R803"  Part="1"
+AR Path="/5A7B753D/59D88845" Ref="R903"  Part="1"
+F 0 "R303" H 3200 3734 45  0000 C CNN
+F 1 "390" H 3200 3650 45  0000 C CNN
+F 2 "yageo:0603" H 3180 3700 20  0001 C CNN
+F 3 "" H 3119 3589 60  0001 C CNN
+F 4 "" H 3519 3989 60  0001 C CNN "1st Source Part Number"
+F 5 "Digikey" H 3419 3889 60  0001 C CNN "1st Source"
+F 6 "RC0603FR-07390RL" H 3319 3789 60  0001 C CNN "Manufacturer Part Number"
+F 7 "YAGEO" H 3219 3689 60  0001 C CNN "Manufacturer"
+	1    3150 3550
+	1    0    0    -1
+$EndComp
+$Comp
+L 1K R?
 U 1 1 5A05950C
 P 2750 3550
@@
 $EndComp
 $Comp
-L icu-rescue:1K R?
+L 1K R?
 U 1 1 5A059568
 P 2750 4100
@@
 $EndComp
 $Comp
-L icu-rescue:DIODE_RS07J-GS18 D302
+L DIODE_RS07J-GS18 D302
 U 1 1 5A2AAF9E
 P 5450 4750
@@
 $EndComp
 $Comp
-L icu-rescue:DIODE_RS07J-GS18 D303
+L DIODE_RS07J-GS18 D303
 U 1 1 5A2AB087
 P 5700 4750
@@
 $EndComp
 $Comp
-L icu-rescue:GND #PWR047
+L GND #PWR047
 U 1 1 5A2AB10F
 P 5550 5150
@@
 $EndComp
 Wire Wire Line
-	5250 3650 5250 3800
+	5250 3650 5250 4000
 Wire Wire Line
 	5250 3800 5100 3800
@@
 Connection ~ 5250 3900
 Wire Wire Line
-	5100 4100 5250 4100
+	5100 4100 5800 4100
 Wire Wire Line
 	5100 4200 5250 4200
@@
 Connection ~ 5250 4100
 Wire Wire Line
-	5100 4400 5250 4400
+	5100 4400 5800 4400
 Wire Wire Line
 	5100 4300 5250 4300
@@
 Connection ~ 5250 4400
 Wire Wire Line
-	2550 3450 2650 3450
-Wire Wire Line
-	2550 4000 2650 4000
-Wire Wire Line
-	2950 3550 2950 4100
-Wire Wire Line
-	2950 4300 3500 4300
+	2550 3450 4300 3450
+Wire Wire Line
+	2550 4000 4300 4000
+Wire Wire Line
+	2950 3550 2950 4450
+Wire Wire Line
+	2950 4300 4300 4300
 Wire Wire Line
 	3050 3550 2950 3550
@@
 Connection ~ 2950 4100
 Wire Wire Line
-	3350 3550 3500 3550
+	3350 3550 4150 3550
+Wire Wire Line
+	3500 3200 3500 3550
 Wire Wire Line
 	3500 3350 2550 3350
@@
 	5700 5050 5700 4950
 Wire Wire Line
-	5450 5050 5550 5050
+	5450 5050 5700 5050
 Wire Wire Line
 	5450 5050 5450 4950
@@
 	4300 3900 4150 3900
 Wire Wire Line
-	4150 3550 4150 3900
+	4150 3550 4150 4100
 Wire Wire Line
 	4300 3450 4300 3800
 $Comp
-L icu-rescue:4.7uF C301
+L 4.7uF C301
 U 1 1 5A708309
 P 3150 3850
@@
 Wire Wire Line
 	3050 3850 3050 3550
+Connection ~ 3050 3550
 Wire Wire Line
 	3350 3850 3350 3550
+Connection ~ 3350 3550
 Wire Wire Line
 	4150 4100 4300 4100
 Connection ~ 4150 3900
-Wire Wire Line
-	5250 3800 5250 3900
-Wire Wire Line
-	5250 3900 5250 4000
-Wire Wire Line
-	5250 4100 5450 4100
-Wire Wire Line
-	5250 4400 5700 4400
-Wire Wire Line
-	2950 4300 2950 4450
-Wire Wire Line
-	2950 4100 2950 4300
-Wire Wire Line
-	3500 3550 4150 3550
-Wire Wire Line
-	2650 3450 4300 3450
-Wire Wire Line
-	2650 4000 4300 4000
-Wire Wire Line
-	5700 4400 5800 4400
-Wire Wire Line
-	5450 4100 5800 4100
-Wire Wire Line
-	5550 5050 5700 5050
-Wire Wire Line
-	4150 3900 4150 4100
-Wire Wire Line
-	3500 3350 3500 3550
-$Comp
-L yageo:1K R603
-U 1 1 5B1E176A
-P 3150 3550
-AR Path="/5A7B4C13/5B1E176A" Ref="R603"  Part="1"
-AR Path="/5A7B2C1B/5B1E176A" Ref="R303"  Part="1"
-AR Path="/5A7B341B/5B1E176A" Ref="R403"  Part="1"
-AR Path="/5A7B3FAD/5B1E176A" Ref="R503"  Part="1"
-AR Path="/5A7B577E/5B1E176A" Ref="R703"  Part="1"
-AR Path="/5A7B753D/5B1E176A" Ref="R803"  Part="1"
-AR Path="/5A7B157A/5B1E176A" Ref="R1003"  Part="1"
-F 0 "R1003" H 3200 3734 45  0000 C CNN
-F 1 "1K" H 3200 3650 45  0000 C CNN
-F 2 "yageo:0603" H 3180 3700 20  0001 C CNN
-F 3 "" H 3119 3589 60  0001 C CNN
-F 4 "" H 3519 3989 60  0001 C CNN "1st Source Part Number"
-F 5 "Digikey" H 3419 3889 60  0001 C CNN "1st Source"
-F 6 "RC0603FR-071KL" H 3319 3789 60  0001 C CNN "Manufacturer Part Number"
-F 7 "YAGEO" H 3219 3689 60  0001 C CNN "Manufacturer"
-	1    3150 3550
-	1    0    0    -1
-$EndComp
-Connection ~ 3350 3550
-Connection ~ 3050 3550
-$Comp
-L usevolt:ZENER_MM3Z3V6T1G D801
-U 1 1 5B753167
-P 3500 3600
-AR Path="/5A7B753D/5B753167" Ref="D801"  Part="1"
-AR Path="/5A7B2C1B/5B753167" Ref="D301"  Part="1"
-AR Path="/5A7B341B/5B753167" Ref="D401"  Part="1"
-AR Path="/5A7B3FAD/5B753167" Ref="D501"  Part="1"
-AR Path="/5A7B4C13/5B753167" Ref="D601"  Part="1"
-AR Path="/5A7B577E/5B753167" Ref="D701"  Part="1"
-AR Path="/5A7B157A/5B753167" Ref="D1001"  Part="1"
-F 0 "D1001" V 3425 3522 45  0000 R CNN
-F 1 "ZENER_MM3Z3V6T1G" H 3775 3975 45  0001 L BNN
-F 2 "usevolt:SOD-323" H 3475 3975 20  0001 C CNN
-F 3 "http://www.mouser.com/ds/2/308/MM3Z2V4T1-D-269162.pdf" H 3850 4175 60  0001 C CNN
-F 4 "Mouser" H 3820 3920 60  0001 C CNN "1st Source"
-F 5 "MM3Z3V6T1G" H 3720 3820 60  0001 C CNN "Manufacturer Part Number"
-F 6 "863-MM3Z3V6T1G" H 3920 4020 60  0001 C CNN "1st Source Part Number"
-F 7 "ON Semiconductor" H 3775 4075 60  0001 C CNN "Manufacturer"
-	1    3500 3600
-	0    -1   -1   0
-$EndComp
-Wire Wire Line
-	3500 3800 3500 4300
-Connection ~ 3500 4300
-Wire Wire Line
-	3500 4300 4300 4300
+$Comp
+L DIODE_RS07J-GS18 D301
+U 1 1 5A7BC689
+P 3700 3200
+AR Path="/5A7B157A/5A7BC689" Ref="D301"  Part="1"
+AR Path="/5A7B341B/5A7BC689" Ref="D501"  Part="1"
+AR Path="/5A7B2C1B/5A7BC689" Ref="D401"  Part="1"
+AR Path="/5A7B3FAD/5A7BC689" Ref="D601"  Part="1"
+AR Path="/5A7B4C13/5A7BC689" Ref="D701"  Part="1"
+AR Path="/5A7B577E/5A7BC689" Ref="D801"  Part="1"
+AR Path="/5A7B753D/5A7BC689" Ref="D901"  Part="1"
+F 0 "D301" H 3650 3340 45  0000 C CNN
+F 1 "DIODE_RS07J-GS18" H 3720 3140 45  0001 L BNN
+F 2 "usevolt:DO219AB" H 3730 3350 20  0001 C CNN
+F 3 "http://www.vishay.com/docs/85742/rs07b.pdf" H 3720 3220 60  0001 C CNN
+F 4 "1864882" H 4320 3820 60  0001 C CNN "2nd Source Part Number"
+F 5 "Digi-Key" H 4020 3520 60  0001 C CNN "1st Source"
+F 6 "Farnell" H 4220 3720 60  0001 C CNN "2nd Source"
+F 7 "RS07J-GS18" H 3920 3420 60  0001 C CNN "Manufacturer Part Number"
+F 8 "RS07J-GS18-ND" H 4120 3620 60  0001 C CNN "1st Source Part Number"
+F 9 "Vishay Semiconductor Diodes Division" H 3820 3320 60  0001 C CNN "Manufacturer"
+	1    3700 3200
+	1    0    0    -1
+$EndComp
+Connection ~ 3500 3350
+$Comp
+L +3V3 #PWR048
+U 1 1 5A7BC750
+P 3900 3100
+AR Path="/5A7B157A/5A7BC750" Ref="#PWR048"  Part="1"
+AR Path="/5A7B341B/5A7BC750" Ref="#PWR020"  Part="1"
+AR Path="/5A7B2C1B/5A7BC750" Ref="#PWR016"  Part="1"
+AR Path="/5A7B3FAD/5A7BC750" Ref="#PWR024"  Part="1"
+AR Path="/5A7B4C13/5A7BC750" Ref="#PWR028"  Part="1"
+AR Path="/5A7B577E/5A7BC750" Ref="#PWR032"  Part="1"
+AR Path="/5A7B753D/5A7BC750" Ref="#PWR036"  Part="1"
+F 0 "#PWR048" H 3900 2950 50  0001 C CNN
+F 1 "+3V3" H 3915 3273 50  0000 C CNN
+F 2 "" H 3900 3100 50  0000 C CNN
+F 3 "" H 3900 3100 50  0000 C CNN
+	1    3900 3100
+	1    0    0    -1
+$EndComp
+Wire Wire Line
+	3900 3100 3900 3200
+Wire Wire Line
+	3900 3200 3800 3200
 $EndSCHEMATC

Commit message: 3.0.0 hw and gerber created
Parts:
- removed D301: DIODE_RS07J-GS18, usevolt:DO219AB, symbol DIODE_RS07J-GS18
- removed R303: 390, yageo:0603, symbol 390
- added D5: ZENER_MM3Z3V6T1G, usevolt:SOD-323, symbol usevolt:ZENER_MM3Z3V6T1G
- added R5: 1K, yageo:0603, symbol yageo:1K
- C301: symbol 4.7uF -> kemet:4.7uF
- D302, D303: symbol DIODE_RS07J-GS18 -> usevolt:DIODE_RS07J-GS18
- R301, R302: symbol 1K -> yageo:1K
- U301: symbol VND5050AJTR-E -> usevolt:VND5050AJTR-E
Connections:
- net GND: now also D5.2, R5.2 (R2)
- net SENSE: now also D5.1, R5.1 (R1)
