File: hw/icu.sch (KiCad schematic (older format))
At the start: 5 parts, among them J101 AMPSEAL_8_POS_VERT_BLACK_SEAL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, J102 AMPSEAL_23_POS_VERT_GRAY_SEAL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

Commit message: hw 1.0 ready to order
Parts:
- removed F102: FUSE_MC36211_350MA, usevolt:FUSE_MC36211, symbol FUSE_MC36211_350MA
- removed R101: R_75OHM, usevolt:1206, symbol R_75OHM
Connections:
- net labels removed: GND
- wire segments 114 -> 109
Other:
- moved on the sheet: J102D, J102E, J102F, J102G, J102H, J102W
Changed lines of the file:
@@
 $Descr A3 16535 11693
 encoding utf-8
-Sheet 1 13
+Sheet 1 14
 Title "ESB version 1"
 Date "2017-02-02"
@@
 $EndSheet
 $Comp
-L +3V3 #PWR104
+L +3V3 #PWR01
 U 1 1 57E93CBF
 P 4900 2050
-F 0 "#PWR104" H 4900 1900 50  0001 C CNN
+F 0 "#PWR01" H 4900 1900 50  0001 C CNN
 F 1 "+3V3" H 4915 2223 50  0000 C CNN
 F 2 "" H 4900 2050 50  0000 C CNN
@@
 $EndComp
 $Comp
-L VDD #PWR102
+L VDD #PWR02
 U 1 1 57E93E22
 P 4400 2050
-F 0 "#PWR102" H 4400 1900 50  0001 C CNN
+F 0 "#PWR02" H 4400 1900 50  0001 C CNN
 F 1 "VDD" H 4417 2223 50  0000 C CNN
 F 2 "" H 4400 2050 50  0000 C CNN
@@
 $EndComp
 $Comp
-L +5V #PWR103
+L +5V #PWR03
 U 1 1 589766AF
 P 4650 2050
-F 0 "#PWR103" H 4650 1900 50  0001 C CNN
+F 0 "#PWR03" H 4650 1900 50  0001 C CNN
 F 1 "+5V" H 4665 2223 50  0000 C CNN
 F 2 "" H 4650 2050 50  0000 C CNN
@@
 $EndComp
 Wire Wire Line
-	1450 2100 1650 2100
-Wire Wire Line
-	1650 2100 3200 2100
+	1450 2100 3200 2100
 Wire Wire Line
 	1450 2400 1650 2400
 Wire Wire Line
-	1650 2100 1650 2400
-Wire Wire Line
-	1650 2400 1650 2850
+	1650 2100 1650 2850
 Connection ~ 1650 2100
 Wire Wire Line
@@
 L AMPSEAL_23_POS_VERT_GRAY_SEALED_1-776228-4 J102
 U 4 1 5A7B03F0
+P 4600 5350
+F 0 "J102" H 4629 5332 45  0000 L CNN
+F 1 "AMPSEAL_23_POS_VERT_GRAY_SEALED_1-776228-4" H 4600 5350 45  0001 L BNN
+F 2 "usevolt:AMPSEAL_23_POS_776200-1" H 4630 5500 20  0001 C CNN
+F 3 "http://www.mouser.com/ds/2/418/NG_CD_776228_C13-672564.pdf" H 4700 5320 60  0001 C CNN
+F 4 "571-1-776228-4" H 5100 5720 60  0001 C CNN "1st Source Part Number"
+F 5 "1-776228-4" H 4900 5520 60  0001 C CNN "Manufacturer Part Number"
+F 6 "Mouser" H 5000 5620 60  0001 C CNN "1st Source"
+F 7 "TE Connectivity" H 4800 5420 60  0001 C CNN "Manufacturer"
+	4    4600 5350
+	-1   0    0    -1
+$EndComp
+$Comp
+L AMPSEAL_23_POS_VERT_GRAY_SEALED_1-776228-4 J102
+U 5 1 5A7B0464
 P 4600 5600
 F 0 "J102" H 4629 5582 45  0000 L CNN
@@
 F 6 "Mouser" H 5000 5870 60  0001 C CNN "1st Source"
 F 7 "TE Connectivity" H 4800 5670 60  0001 C CNN "Manufacturer"
-	4    4600 5600
-	-1   0    0    -1
-$EndComp
-$Comp
-L AMPSEAL_23_POS_VERT_GRAY_SEALED_1-776228-4 J102
-U 5 1 5A7B0464
+	5    4600 5600
+	-1   0    0    -1
+$EndComp
+$Comp
+L AMPSEAL_23_POS_VERT_GRAY_SEALED_1-776228-4 J102
+U 6 1 5A7B04DA
 P 4600 6000
 F 0 "J102" H 4629 5982 45  0000 L CNN
@@
 F 6 "Mouser" H 5000 6270 60  0001 C CNN "1st Source"
 F 7 "TE Connectivity" H 4800 6070 60  0001 C CNN "Manufacturer"
-	5    4600 6000
-	-1   0    0    -1
-$EndComp
-$Comp
-L AMPSEAL_23_POS_VERT_GRAY_SEALED_1-776228-4 J102
-U 6 1 5A7B04DA
+	6    4600 6000
+	-1   0    0    -1
+$EndComp
+$Comp
+L AMPSEAL_23_POS_VERT_GRAY_SEALED_1-776228-4 J102
+U 7 1 5A7B0552
 P 4600 6400
 F 0 "J102" H 4629 6382 45  0000 L CNN
@@
 F 6 "Mouser" H 5000 6670 60  0001 C CNN "1st Source"
 F 7 "TE Connectivity" H 4800 6470 60  0001 C CNN "Manufacturer"
-	6    4600 6400
-	-1   0    0    -1
-$EndComp
-$Comp
-L AMPSEAL_23_POS_VERT_GRAY_SEALED_1-776228-4 J102
-U 7 1 5A7B0552
-P 1700 7050
-F 0 "J102" H 1729 7032 45  0000 L CNN
-F 1 "AMPSEAL_23_POS_VERT_GRAY_SEALED_1-776228-4" H 1700 7050 45  0001 L BNN
-F 2 "usevolt:AMPSEAL_23_POS_776200-1" H 1730 7200 20  0001 C CNN
-F 3 "http://www.mouser.com/ds/2/418/NG_CD_776228_C13-672564.pdf" H 1800 7020 60  0001 C CNN
-F 4 "571-1-776228-4" H 2200 7420 60  0001 C CNN "1st Source Part Number"
-F 5 "1-776228-4" H 2000 7220 60  0001 C CNN "Manufacturer Part Number"
-F 6 "Mouser" H 2100 7320 60  0001 C CNN "1st Source"
-F 7 "TE Connectivity" H 1900 7120 60  0001 C CNN "Manufacturer"
-	7    1700 7050
+	7    4600 6400
 	-1   0    0    -1
 $EndComp
@@
 L AMPSEAL_23_POS_VERT_GRAY_SEALED_1-776228-4 J102
 U 8 1 5A7B05CC
-P 1700 5850
-F 0 "J102" H 1729 5832 45  0000 L CNN
-F 1 "AMPSEAL_23_POS_VERT_GRAY_SEALED_1-776228-4" H 1700 5850 45  0001 L BNN
-F 2 "usevolt:AMPSEAL_23_POS_776200-1" H 1730 6000 20  0001 C CNN
-F 3 "http://www.mouser.com/ds/2/418/NG_CD_776228_C13-672564.pdf" H 1800 5820 60  0001 C CNN
-F 4 "571-1-776228-4" H 2200 6220 60  0001 C CNN "1st Source Part Number"
-F 5 "1-776228-4" H 2000 6020 60  0001 C CNN "Manufacturer Part Number"
-F 6 "Mouser" H 2100 6120 60  0001 C CNN "1st Source"
-F 7 "TE Connectivity" H 1900 5920 60  0001 C CNN "Manufacturer"
-	8    1700 5850
+P 4600 6800
+F 0 "J102" H 4629 6782 45  0000 L CNN
+F 1 "AMPSEAL_23_POS_VERT_GRAY_SEALED_1-776228-4" H 4600 6800 45  0001 L BNN
+F 2 "usevolt:AMPSEAL_23_POS_776200-1" H 4630 6950 20  0001 C CNN
+F 3 "http://www.mouser.com/ds/2/418/NG_CD_776228_C13-672564.pdf" H 4700 6770 60  0001 C CNN
+F 4 "571-1-776228-4" H 5100 7170 60  0001 C CNN "1st Source Part Number"
+F 5 "1-776228-4" H 4900 6970 60  0001 C CNN "Manufacturer Part Number"
+F 6 "Mouser" H 5000 7070 60  0001 C CNN "1st Source"
+F 7 "TE Connectivity" H 4800 6870 60  0001 C CNN "Manufacturer"
+	8    4600 6800
 	-1   0    0    -1
 $EndComp
@@
 L AMPSEAL_23_POS_VERT_GRAY_SEALED_1-776228-4 J102
 U 23 1 5A7B103A
-P 1700 6750
-F 0 "J102" H 1729 6732 45  0000 L CNN
-F 1 "AMPSEAL_23_POS_VERT_GRAY_SEALED_1-776228-4" H 1700 6750 45  0001 L BNN
-F 2 "usevolt:AMPSEAL_23_POS_776200-1" H 1730 6900 20  0001 C CNN
-F 3 "http://www.mouser.com/ds/2/418/NG_CD_776228_C13-672564.pdf" H 1800 6720 60  0001 C CNN
-F 4 "571-1-776228-4" H 2200 7120 60  0001 C CNN "1st Source Part Number"
-F 5 "1-776228-4" H 2000 6920 60  0001 C CNN "Manufacturer Part Number"
-F 6 "Mouser" H 2100 7020 60  0001 C CNN "1st Source"
-F 7 "TE Connectivity" H 1900 6820 60  0001 C CNN "Manufacturer"
-	23   1700 6750
+P 1700 5850
+F 0 "J102" H 1729 5832 45  0000 L CNN
+F 1 "AMPSEAL_23_POS_VERT_GRAY_SEALED_1-776228-4" H 1700 5850 45  0001 L BNN
+F 2 "usevolt:AMPSEAL_23_POS_776200-1" H 1730 6000 20  0001 C CNN
+F 3 "http://www.mouser.com/ds/2/418/NG_CD_776228_C13-672564.pdf" H 1800 5820 60  0001 C CNN
+F 4 "571-1-776228-4" H 2200 6220 60  0001 C CNN "1st Source Part Number"
+F 5 "1-776228-4" H 2000 6020 60  0001 C CNN "Manufacturer Part Number"
+F 6 "Mouser" H 2100 6120 60  0001 C CNN "1st Source"
+F 7 "TE Connectivity" H 1900 5920 60  0001 C CNN "Manufacturer"
+	23   1700 5850
 	-1   0    0    -1
 $EndComp
@@
 F29 "AIN2" I L 7200 6000 60
 F30 "AIN3" I L 7200 6400 60
+F31 "AIN4" I L 7200 6800 60
+F32 "DIN4" I L 7200 5350 60
 $EndSheet
 Wire Wire Line
@@
 5V_OUT
 $Comp
-L +5V #PWR101
+L +5V #PWR04
 U 1 1 5A7DBD62
 P 2800 5650
-F 0 "#PWR101" H 2800 5500 50  0001 C CNN
+F 0 "#PWR04" H 2800 5500 50  0001 C CNN
 F 1 "+5V" H 2815 5823 50  0000 C CNN
 F 2 "" H 2800 5650 50  0000 C CNN
@@
 Wire Wire Line
 	7200 5600 6000 5600
-$Comp
-L R_75OHM R101
-U 1 1 5A7EE4F1
-P 2300 7050
-F 0 "R101" H 2300 7287 60  0000 C CNN
-F 1 "R_75OHM" H 2300 7181 60  0000 C CNN
-F 2 "usevolt:1206" H 2200 7150 60  0001 C CNN
-F 3 "http://www.farnell.com/datasheets/2158849.pdf?_ga=1.165170815.1561825231.1484148445" H 2300 7250 60  0001 C CNN
-F 4 "1100161" H 2700 7650 60  0001 C CNN "1st Source Part Number"
-F 5 "WCR1206-75RFI" H 2500 7450 60  0001 C CNN "Manufacturer Part Number"
-F 6 "Farnell" H 2600 7550 60  0001 C CNN "1st Source"
-F 7 "WELWYN" H 2400 7350 60  0001 C CNN "Manufacturer"
-	1    2300 7050
-	1    0    0    -1
-$EndComp
-Wire Wire Line
-	2100 7050 1800 7050
-$Comp
-L GND #PWR106
-U 1 1 5A7EFDA7
-P 2750 7250
-F 0 "#PWR106" H 2750 7000 50  0001 C CNN
-F 1 "GND" H 2755 7077 50  0000 C CNN
-F 2 "" H 2750 7250 50  0000 C CNN
-F 3 "" H 2750 7250 50  0000 C CNN
-	1    2750 7250
-	1    0    0    -1
-$EndComp
-Wire Wire Line
-	2750 7250 2750 7050
-Wire Wire Line
-	2750 7050 2500 7050
-$Comp
-L FUSE_MC36211_350MA F102
-U 1 1 5A7F657D
-P 2750 6500
-F 0 "F102" V 2708 6578 45  0000 L CNN
-F 1 "FUSE_MC36211_350MA" V 2792 6578 45  0000 L CNN
-F 2 "usevolt:FUSE_MC36211" H 2780 6650 20  0001 C CNN
-F 3 "http://www.farnell.com/datasheets/1678471.pdf?_ga=1.218604761.1948984246.1460023966" H 2870 6520 60  0001 C CNN
-F 4 "Farnell" H 3170 6820 60  0001 C CNN "1st Source"
-F 5 "MC36211" H 3070 6720 60  0001 C CNN "Manufacturer Part Number"
-F 6 "MC36211" H 3270 6920 60  0001 C CNN "1st Source Part Number"
-F 7 "Multicomp" H 2970 6620 60  0001 C CNN "Manufacturer"
-	1    2750 6500
-	0    1    1    0
-$EndComp
-Wire Wire Line
-	2750 6700 2750 6750
-Wire Wire Line
-	2750 6750 1800 6750
-$Comp
-L VDD #PWR105
-U 1 1 5A7F6A4F
-P 2750 6250
-F 0 "#PWR105" H 2750 6100 50  0001 C CNN
-F 1 "VDD" H 2767 6423 50  0000 C CNN
-F 2 "" H 2750 6250 50  0000 C CNN
-F 3 "" H 2750 6250 50  0000 C CNN
-	1    2750 6250
-	1    0    0    -1
-$EndComp
-Wire Wire Line
-	2750 6250 2750 6300
+$Sheet
+S 5100 6700 900  200
+U 5A8C5348
+F0 "Sheet5A8C5347" 60
+F1 "ain.sch" 60
+F2 "VOUT" O R 6000 6800 60
+F3 "VIN" I L 5100 6800 60
+$EndSheet
+Wire Wire Line
+	5100 6800 4700 6800
+Wire Wire Line
+	7200 5350 4700 5350
+Wire Wire Line
+	6000 6800 7200 6800
 $EndSCHEMATC

Commit message: 3.0.0 hw and gerber created
Parts:
- F101: symbol FUSE_MC36211_350MA -> usevolt:FUSE_MC36211_350MA
- J101: symbol AMPSEAL_8_POS_VERT_BLACK_SEALED_1-776276-1 -> usevolt:AMPSEAL_8_POS_VERT_BLACK_SEALED_1-776276-1
- J102: symbol AMPSEAL_23_POS_VERT_GRAY_SEALED_1-776228-4 -> usevolt:AMPSEAL_23_POS_VERT_GRAY_SEALED_1-776228-4
Changed lines of the file:
@@
-EESchema Schematic File Version 2
-LIBS:kemet
-LIBS:usevolt
-LIBS:wurth_elektronik_LED
-LIBS:power
-LIBS:yageo
+EESchema Schematic File Version 4
 LIBS:icu-cache
 EELAYER 26 0
@@
 $EndSheet
 $Comp
-L +3V3 #PWR01
+L power:+3V3 #PWR01
 U 1 1 57E93CBF
 P 4900 2050
@@
 $EndComp
 $Comp
-L VDD #PWR02
+L power:VDD #PWR02
 U 1 1 57E93E22
 P 4400 2050
@@
 $EndComp
 $Comp
-L +5V #PWR03
+L power:+5V #PWR03
 U 1 1 589766AF
 P 4650 2050
@@
 	4650 2250 4300 2250
 $Comp
-L AMPSEAL_8_POS_VERT_BLACK_SEALED_1-776276-1 J101
+L usevolt:AMPSEAL_8_POS_VERT_BLACK_SEALED_1-776276-1 J101
 U 1 1 5A79A3F3
 P 1350 2100
@@
 $EndComp
 $Comp
-L AMPSEAL_8_POS_VERT_BLACK_SEALED_1-776276-1 J101
+L usevolt:AMPSEAL_8_POS_VERT_BLACK_SEALED_1-776276-1 J101
 U 2 1 5A79A545
 P 1350 2250
@@
 $EndComp
 $Comp
-L AMPSEAL_8_POS_VERT_BLACK_SEALED_1-776276-1 J101
+L usevolt:AMPSEAL_8_POS_VERT_BLACK_SEALED_1-776276-1 J101
 U 3 1 5A79A8B7
 P 1350 2400
@@
 $EndComp
 $Comp
-L AMPSEAL_8_POS_VERT_BLACK_SEALED_1-776276-1 J101
+L usevolt:AMPSEAL_8_POS_VERT_BLACK_SEALED_1-776276-1 J101
 U 4 1 5A79A9C7
 P 1350 2550
@@
 $EndComp
 $Comp
-L AMPSEAL_8_POS_VERT_BLACK_SEALED_1-776276-1 J101
+L usevolt:AMPSEAL_8_POS_VERT_BLACK_SEALED_1-776276-1 J101
 U 5 1 5A79AADD
 P 1350 2700
@@
 $EndComp
 $Comp
-L AMPSEAL_8_POS_VERT_BLACK_SEALED_1-776276-1 J101
+L usevolt:AMPSEAL_8_POS_VERT_BLACK_SEALED_1-776276-1 J101
 U 6 1 5A79AD45
 P 1350 2850
@@
 $EndComp
 $Comp
-L AMPSEAL_8_POS_VERT_BLACK_SEALED_1-776276-1 J101
+L usevolt:AMPSEAL_8_POS_VERT_BLACK_SEALED_1-776276-1 J101
 U 7 1 5A79AE65
 P 1350 3000
@@
 $EndComp
 $Comp
-L AMPSEAL_8_POS_VERT_BLACK_SEALED_1-776276-1 J101
+L usevolt:AMPSEAL_8_POS_VERT_BLACK_SEALED_1-776276-1 J101
 U 8 1 5A79AF81
 P 1350 3150
@@
 $EndComp
 Wire Wire Line
-	1450 2100 3200 2100
+	1450 2100 1650 2100
 Wire Wire Line
 	1450 2400 1650 2400
 Wire Wire Line
-	1650 2100 1650 2850
+	1650 2100 1650 2400
 Connection ~ 1650 2100
 Wire Wire Line
@@
 	5800 4550 7200 4550
 $Comp
-L AMPSEAL_23_POS_VERT_GRAY_SEALED_1-776228-4 J102
+L usevolt:AMPSEAL_23_POS_VERT_GRAY_SEALED_1-776228-4 J102
 U 1 1 5A7B0192
 P 4600 5050
@@
 $EndComp
 $Comp
-L AMPSEAL_23_POS_VERT_GRAY_SEALED_1-776228-4 J102
+L usevolt:AMPSEAL_23_POS_VERT_GRAY_SEALED_1-776228-4 J102
 U 2 1 5A7B0214
 P 4600 5150
@@
 $EndComp
 $Comp
-L AMPSEAL_23_POS_VERT_GRAY_SEALED_1-776228-4 J102
+L usevolt:AMPSEAL_23_POS_VERT_GRAY_SEALED_1-776228-4 J102
 U 3 1 5A7B037A
 P 4600 5250
@@
 $EndComp
 $Comp
-L AMPSEAL_23_POS_VERT_GRAY_SEALED_1-776228-4 J102
+L usevolt:AMPSEAL_23_POS_VERT_GRAY_SEALED_1-776228-4 J102
 U 4 1 5A7B03F0
 P 4600 5350
@@
 $EndComp
 $Comp
-L AMPSEAL_23_POS_VERT_GRAY_SEALED_1-776228-4 J102
+L usevolt:AMPSEAL_23_POS_VERT_GRAY_SEALED_1-776228-4 J102
 U 5 1 5A7B0464
 P 4600 5600
@@
 $EndComp
 $Comp
-L AMPSEAL_23_POS_VERT_GRAY_SEALED_1-776228-4 J102
+L usevolt:AMPSEAL_23_POS_VERT_GRAY_SEALED_1-776228-4 J102
 U 6 1 5A7B04DA
 P 4600 6000
@@
 $EndComp
 $Comp
-L AMPSEAL_23_POS_VERT_GRAY_SEALED_1-776228-4 J102
+L usevolt:AMPSEAL_23_POS_VERT_GRAY_SEALED_1-776228-4 J102
 U 7 1 5A7B0552
 P 4600 6400
@@
 $EndComp
 $Comp
-L AMPSEAL_23_POS_VERT_GRAY_SEALED_1-776228-4 J102
+L usevolt:AMPSEAL_23_POS_VERT_GRAY_SEALED_1-776228-4 J102
 U 8 1 5A7B05CC
 P 4600 6800
@@
 $EndComp
 $Comp
-L AMPSEAL_23_POS_VERT_GRAY_SEALED_1-776228-4 J102
+L usevolt:AMPSEAL_23_POS_VERT_GRAY_SEALED_1-776228-4 J102
 U 9 1 5A7B0648
 P 12750 3600
@@
 $EndComp
 $Comp
-L AMPSEAL_23_POS_VERT_GRAY_SEALED_1-776228-4 J102
+L usevolt:AMPSEAL_23_POS_VERT_GRAY_SEALED_1-776228-4 J102
 U 10 1 5A7B075E
 P 12750 4200
@@
 $EndComp
 $Comp
-L AMPSEAL_23_POS_VERT_GRAY_SEALED_1-776228-4 J102
+L usevolt:AMPSEAL_23_POS_VERT_GRAY_SEALED_1-776228-4 J102
 U 11 1 5A7B07EA
 P 12750 4800
@@
 $EndComp
 $Comp
-L AMPSEAL_23_POS_VERT_GRAY_SEALED_1-776228-4 J102
+L usevolt:AMPSEAL_23_POS_VERT_GRAY_SEALED_1-776228-4 J102
 U 12 1 5A7B086C
 P 12750 5400
@@
 $EndComp
 $Comp
-L AMPSEAL_23_POS_VERT_GRAY_SEALED_1-776228-4 J102
+L usevolt:AMPSEAL_23_POS_VERT_GRAY_SEALED_1-776228-4 J102
 U 13 1 5A7B08F0
 P 12750 6000
@@
 $EndComp
 $Comp
-L AMPSEAL_23_POS_VERT_GRAY_SEALED_1-776228-4 J102
+L usevolt:AMPSEAL_23_POS_VERT_GRAY_SEALED_1-776228-4 J102
 U 14 1 5A7B0976
 P 12750 6600
@@
 $EndComp
 $Comp
-L AMPSEAL_23_POS_VERT_GRAY_SEALED_1-776228-4 J102
+L usevolt:AMPSEAL_23_POS_VERT_GRAY_SEALED_1-776228-4 J102
 U 15 1 5A7B09FE
 P 12750 7200
@@
 $EndComp
 $Comp
-L AMPSEAL_23_POS_VERT_GRAY_SEALED_1-776228-4 J102
+L usevolt:AMPSEAL_23_POS_VERT_GRAY_SEALED_1-776228-4 J102
 U 16 1 5A7B0A88
 P 12750 3800
@@
 $EndComp
 $Comp
-L AMPSEAL_23_POS_VERT_GRAY_SEALED_1-776228-4 J102
+L usevolt:AMPSEAL_23_POS_VERT_GRAY_SEALED_1-776228-4 J102
 U 17 1 5A7B0B14
 P 12750 4400
@@
 $EndComp
 $Comp
-L AMPSEAL_23_POS_VERT_GRAY_SEALED_1-776228-4 J102
+L usevolt:AMPSEAL_23_POS_VERT_GRAY_SEALED_1-776228-4 J102
 U 18 1 5A7B0C28
 P 12750 5000
@@
 $EndComp
 $Comp
-L AMPSEAL_23_POS_VERT_GRAY_SEALED_1-776228-4 J102
+L usevolt:AMPSEAL_23_POS_VERT_GRAY_SEALED_1-776228-4 J102
 U 19 1 5A7B0CB4
 P 12750 5600
@@
 $EndComp
 $Comp
-L AMPSEAL_23_POS_VERT_GRAY_SEALED_1-776228-4 J102
+L usevolt:AMPSEAL_23_POS_VERT_GRAY_SEALED_1-776228-4 J102
 U 20 1 5A7B0DD2
 P 12750 6200
@@
 $EndComp
 $Comp
-L AMPSEAL_23_POS_VERT_GRAY_SEALED_1-776228-4 J102
+L usevolt:AMPSEAL_23_POS_VERT_GRAY_SEALED_1-776228-4 J102
 U 21 1 5A7B0F0C
 P 12750 6800
@@
 $EndComp
 $Comp
-L AMPSEAL_23_POS_VERT_GRAY_SEALED_1-776228-4 J102
+L usevolt:AMPSEAL_23_POS_VERT_GRAY_SEALED_1-776228-4 J102
 U 22 1 5A7B0FA2
 P 12750 7400
@@
 $EndComp
 $Comp
-L AMPSEAL_23_POS_VERT_GRAY_SEALED_1-776228-4 J102
+L usevolt:AMPSEAL_23_POS_VERT_GRAY_SEALED_1-776228-4 J102
 U 23 1 5A7B103A
 P 1700 5850
@@
 	12450 4200 12650 4200
 $Comp
-L FUSE_MC36211_350MA F101
+L usevolt:FUSE_MC36211_350MA F101
 U 1 1 5A7D8C08
 P 2400 5850
@@
 5V_OUT
 $Comp
-L +5V #PWR04
+L power:+5V #PWR04
 U 1 1 5A7DBD62
 P 2800 5650
@@
 Wire Wire Line
 	6000 6800 7200 6800
+Wire Wire Line
+	1650 2100 3200 2100
+Wire Wire Line
+	1650 2400 1650 2850
 $EndSCHEMATC

Commit message: 3.3 pcb created
Connections:
- net Sheet5A7E34B9/VIN is gone; now on net SENSORVDD_OUT: J102.7 (S)
- net Sheet5A8C5347/VIN is gone; now on net SENSORVDD_OUT: J102.8 (S)
- net +5V: no longer F101.P$1
- net VDD: now also F101.P$1
- net 5V_OUT renamed SENSORVDD_OUT
Other:
- moved on the sheet: J102G, J102H
Changed lines of the file:
@@
 $Descr A3 16535 11693
 encoding utf-8
-Sheet 1 14
+Sheet 1 12
 Title "ESB version 1"
 Date "2017-02-02"
@@
 L usevolt:AMPSEAL_23_POS_VERT_GRAY_SEALED_1-776228-4 J102
 U 7 1 5A7B0552
-P 4600 6400
-F 0 "J102" H 4629 6382 45  0000 L CNN
-F 1 "AMPSEAL_23_POS_VERT_GRAY_SEALED_1-776228-4" H 4600 6400 45  0001 L BNN
-F 2 "usevolt:AMPSEAL_23_POS_776200-1" H 4630 6550 20  0001 C CNN
-F 3 "http://www.mouser.com/ds/2/418/NG_CD_776228_C13-672564.pdf" H 4700 6370 60  0001 C CNN
-F 4 "571-1-776228-4" H 5100 6770 60  0001 C CNN "1st Source Part Number"
-F 5 "1-776228-4" H 4900 6570 60  0001 C CNN "Manufacturer Part Number"
-F 6 "Mouser" H 5000 6670 60  0001 C CNN "1st Source"
-F 7 "TE Connectivity" H 4800 6470 60  0001 C CNN "Manufacturer"
-	7    4600 6400
+P 1700 6000
+F 0 "J102" H 1729 5982 45  0000 L CNN
+F 1 "AMPSEAL_23_POS_VERT_GRAY_SEALED_1-776228-4" H 1700 6000 45  0001 L BNN
+F 2 "usevolt:AMPSEAL_23_POS_776200-1" H 1730 6150 20  0001 C CNN
+F 3 "http://www.mouser.com/ds/2/418/NG_CD_776228_C13-672564.pdf" H 1800 5970 60  0001 C CNN
+F 4 "571-1-776228-4" H 2200 6370 60  0001 C CNN "1st Source Part Number"
+F 5 "1-776228-4" H 2000 6170 60  0001 C CNN "Manufacturer Part Number"
+F 6 "Mouser" H 2100 6270 60  0001 C CNN "1st Source"
+F 7 "TE Connectivity" H 1900 6070 60  0001 C CNN "Manufacturer"
+	7    1700 6000
 	-1   0    0    -1
 $EndComp
@@
 L usevolt:AMPSEAL_23_POS_VERT_GRAY_SEALED_1-776228-4 J102
 U 8 1 5A7B05CC
-P 4600 6800
-F 0 "J102" H 4629 6782 45  0000 L CNN
-F 1 "AMPSEAL_23_POS_VERT_GRAY_SEALED_1-776228-4" H 4600 6800 45  0001 L BNN
-F 2 "usevolt:AMPSEAL_23_POS_776200-1" H 4630 6950 20  0001 C CNN
-F 3 "http://www.mouser.com/ds/2/418/NG_CD_776228_C13-672564.pdf" H 4700 6770 60  0001 C CNN
-F 4 "571-1-776228-4" H 5100 7170 60  0001 C CNN "1st Source Part Number"
-F 5 "1-776228-4" H 4900 6970 60  0001 C CNN "Manufacturer Part Number"
-F 6 "Mouser" H 5000 7070 60  0001 C CNN "1st Source"
-F 7 "TE Connectivity" H 4800 6870 60  0001 C CNN "Manufacturer"
-	8    4600 6800
+P 1700 6150
+F 0 "J102" H 1729 6132 45  0000 L CNN
+F 1 "AMPSEAL_23_POS_VERT_GRAY_SEALED_1-776228-4" H 1700 6150 45  0001 L BNN
+F 2 "usevolt:AMPSEAL_23_POS_776200-1" H 1730 6300 20  0001 C CNN
+F 3 "http://www.mouser.com/ds/2/418/NG_CD_776228_C13-672564.pdf" H 1800 6120 60  0001 C CNN
+F 4 "571-1-776228-4" H 2200 6520 60  0001 C CNN "1st Source Part Number"
+F 5 "1-776228-4" H 2000 6320 60  0001 C CNN "Manufacturer Part Number"
+F 6 "Mouser" H 2100 6420 60  0001 C CNN "1st Source"
+F 7 "TE Connectivity" H 1900 6220 60  0001 C CNN "Manufacturer"
+	8    1700 6150
 	-1   0    0    -1
 $EndComp
@@
 	1800 5850 2200 5850
 Text Label 2200 5850 2    60   ~ 0
-5V_OUT
-$Comp
-L power:+5V #PWR04
-U 1 1 5A7DBD62
-P 2800 5650
-F 0 "#PWR04" H 2800 5500 50  0001 C CNN
-F 1 "+5V" H 2815 5823 50  0000 C CNN
-F 2 "" H 2800 5650 50  0000 C CNN
-F 3 "" H 2800 5650 50  0000 C CNN
-	1    2800 5650
-	-1   0    0    -1
-$EndComp
+SENSORVDD_OUT
 Wire Wire Line
 	2800 5650 2800 5850
@@
 F3 "VIN" I L 5100 6000 60
 $EndSheet
-$Sheet
-S 5100 6300 900  200
-U 5A7E34BA
-F0 "Sheet5A7E34B9" 60
-F1 "ain.sch" 60
-F2 "VOUT" O R 6000 6400 60
-F3 "VIN" I L 5100 6400 60
-$EndSheet
 Wire Wire Line
 	4700 5600 5100 5600
@@
 	5100 6000 4700 6000
 Wire Wire Line
-	4700 6400 5100 6400
-Wire Wire Line
 	4700 5050 7200 5050
 Wire Wire Line
@@
 	4700 5250 7200 5250
 Wire Wire Line
-	7200 6400 6000 6400
-Wire Wire Line
 	6000 6000 7200 6000
 Wire Wire Line
 	7200 5600 6000 5600
-$Sheet
-S 5100 6700 900  200
-U 5A8C5348
-F0 "Sheet5A8C5347" 60
-F1 "ain.sch" 60
-F2 "VOUT" O R 6000 6800 60
-F3 "VIN" I L 5100 6800 60
-$EndSheet
-Wire Wire Line
-	5100 6800 4700 6800
 Wire Wire Line
 	7200 5350 4700 5350
 Wire Wire Line
-	6000 6800 7200 6800
-Wire Wire Line
 	1650 2100 3200 2100
 Wire Wire Line
 	1650 2400 1650 2850
+$Comp
+L power:VDD #PWR0101
+U 1 1 5C49CD9F
+P 2800 5650
+F 0 "#PWR0101" H 2800 5500 50  0001 C CNN
+F 1 "VDD" H 2817 5823 50  0000 C CNN
+F 2 "" H 2800 5650 50  0000 C CNN
+F 3 "" H 2800 5650 50  0000 C CNN
+	1    2800 5650
+	1    0    0    -1
+$EndComp
+Wire Wire Line
+	1800 6000 2200 6000
+Wire Wire Line
+	2200 6000 2200 5850
+Connection ~ 2200 5850
+Wire Wire Line
+	1800 6150 2200 6150
+Wire Wire Line
+	2200 6150 2200 6000
+Connection ~ 2200 6000
 $EndSCHEMATC

Commit message: 3.4.0 pcb created
Connections:
- net Power supply/GND: now also J101.8 (S)
Changed lines of the file:
@@
 Connection ~ 1650 2400
 Wire Wire Line
-	1450 2250 2850 2250
+	1450 2250 1750 2250
 Wire Wire Line
 	2850 2250 2850 2800
@@
 	2200 6150 2200 6000
 Connection ~ 2200 6000
+Wire Wire Line
+	1750 2250 1750 3150
+Wire Wire Line
+	1750 3150 1450 3150
+Connection ~ 1750 2250
+Wire Wire Line
+	1750 2250 2850 2250
 $EndSCHEMATC
