File: hw/icu.kicad_pcb (KiCad board)
At the start: 2 copper layers, 60 x 90 mm, 99 parts, among them J1001 ARM_JTAG_SWD_HEADER_10_PINSMD, J101 AMPSEAL_8_POS_VERT_BLACK_SEAL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, J102 AMPSEAL_23_POS_VERT_GRAY_SEAL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, U1001 MCP2551_SOIC8, U1002 LPC1549JBD64, U301 VND5050AJTR-E, U401 VND5050AJTR-E, U501 VND5050AJTR-E, U601 VND5050AJTR-E, U701 VND5050AJTR-E, U901 VND5050AJTR-E, X1001 XTAL_7A-12.000MAAJ-T

Commit message: 3.3 pcb created
Parts:
- removed D1301, D1401: DIODE_RS07J-GS18, usevolt:DO219AB
- removed R1301, R1401: 10K, yageo:0603
- removed R1302, R1402: 20K, yageo:0603
- added C801: 4.7uF, kemet:0603, F.Cu at (183.4, 93.8)
- added D5: ZENER_MM3Z3V6T1G, usevolt:SOD-323, F.Cu at (180.8, 97.8)
- added D802: DIODE_RS07J-GS18, usevolt:DO219AB, F.Cu at (183.2, 81.2)
- added D803: DIODE_RS07J-GS18, usevolt:DO219AB, F.Cu at (178.8, 81.2)
- added R5: 1K, yageo:0603, F.Cu at (181.8, 93.8)
- added R801: 1K, yageo:0603, F.Cu at (180.2, 93.8)
- added R802: 1K, yageo:0603, F.Cu at (178.6, 93.8)
- added U801: VND5050AJTR-E, usevolt:PowerSSO-12, F.Cu at (180.9, 87.8)
Connections:
- F101 pad P$2: /12V_OUT -> /SENSORVDD_OUT
- J102 pad 14: /12V_OUT -> /Sheet5A7B577D/OUT1
- J102 pad 21: /12V_OUT -> /Sheet5A7B577D/OUT2
- J102 pad 23: /12V_OUT -> /SENSORVDD_OUT
- J102 pad 7: /Sheet5A7E34B9/VIN -> /SENSORVDD_OUT
- J102 pad 8: /Sheet5A8C5347/VIN -> /SENSORVDD_OUT
- U1002 pad P$11: Net-(U1002-PadP$11) -> /lpc1549/OUT6_SENSE
- U1002 pad P$19: Net-(U1002-PadP$19) -> /Sheet5A7B577D/IN1
- U1002 pad P$24: Net-(U1002-PadP$24) -> /Sheet5A7B577D/IN2
- U1002 pad P$3: /lpc1549/AIN4 -> Net-(U1002-PadP$3)
- U1002 pad P$4: /lpc1549/AIN3 -> Net-(U1002-PadP$4)
Routing:
- net /lpc1549/AIN4: track 117.1 -> 0.00 mm, vias 2 -> 0
- net /lpc1549/AIN3: track 108.9 -> 0.00 mm, vias 2 -> 0
- net /lpc1549/OUT6_SENSE: track 0.00 -> 61.1 mm, vias 0 -> 2
- net /Sheet5A7B577D/IN1: track 0.00 -> 49.9 mm, vias 0 -> 2
- net /Sheet5A7B577D/IN2: track 0.00 -> 43.2 mm, vias 0 -> 2
- net /Sheet5A7B577D/OUT1: track 0.00 -> 25.6 mm
- net /Sheet5A7B577D/OUT2: track 0.00 -> 21.7 mm
- net /12V_OUT: track 20.6 -> 0.00 mm
- net GND: track 662.8 -> 681.7 mm, vias 93 -> 96
- net /SENSORVDD_OUT: track 0.00 -> 17.2 mm
- net +3V3: track 177.2 -> 169.1 mm
- net VDD: track 20.7 -> 25.0 mm
- net /Sheet5A8C5347/VIN: track 3.69 -> 0.00 mm
- net /Sheet5A7E34B9/VIN: track 3.45 -> 0.00 mm
Other:
- board text added: "UW ICU 3.3 Usevolt Oy"
- board text removed: "UW ISB 3.2 Usevolt Oy"

Commit message: 3.4.0 pcb created
Connections:
- J101 pad 8: Net-(J101-Pad8) -> GND

Commit message: small updates on schematic
Routing:
- net GND: track 681.7 -> 683.1 mm
